Commit message: minor changes

File: vizzy_description/robots/exp.urdf (robot description, URDF)
Before this commit: robot vizzy-description, 18 links, 17 joints
Links:
- link b_wheel_base_link: geometry collision mesh filename=package://vizzy_description/meshes/Back.dae; visual mesh filename=package://vizzy_description/meshes/Back.dae
- link b_wheel_link: geometry collision mesh filename=package://vizzy_description/meshes/B_W.dae; visual mesh filename=package://vizzy_description/meshes/B_W.dae
- link base_link: geometry collision mesh filename=package://vizzy_description/meshes/Segway.dae; visual mesh filename=package://vizzy_description/meshes/Segway.dae
- link f_wheel_base_link: geometry collision mesh filename=package://vizzy_description/meshes/Front.dae; visual mesh filename=package://vizzy_description/meshes/Front.dae
- link f_wheel_link: geometry collision mesh filename=package://vizzy_description/meshes/F_W.dae; visual mesh filename=package://vizzy_description/meshes/F_W.dae
- link l_wheel_link: geometry collision mesh filename=package://vizzy_description/meshes/Right.dae; visual mesh filename=package://vizzy_description/meshes/Right.dae
- link r_elbow_flection_link: geometry collision mesh filename=package://vizzy_description/meshes/M4R.dae; visual mesh filename=package://vizzy_description/meshes/M4R.dae
- link r_forearm_pronation_link: geometry collision mesh filename=package://vizzy_description/meshes/M5R.dae; visual mesh filename=package://vizzy_description/meshes/M5R.dae
- link r_shoulder_abduction_link: geometry collision mesh filename=package://vizzy_description/meshes/M2R.dae; visual mesh filename=package://vizzy_description/meshes/M2R.dae
- link r_shoulder_flection_link: geometry collision mesh filename=package://vizzy_description/meshes/M1R.dae; visual mesh filename=package://vizzy_description/meshes/M1R.dae
- link r_shoulder_rotation_link: geometry collision mesh filename=package://vizzy_description/meshes/M3R.dae; visual mesh filename=package://vizzy_description/meshes/M3R.dae
- link r_shoulder_scapula_link: geometry collision mesh filename=package://vizzy_description/meshes/M0R.dae; visual mesh filename=package://vizzy_description/meshes/M0R.dae
- link r_wheel_link: geometry collision mesh filename=package://vizzy_description/meshes/Left.dae; visual mesh filename=package://vizzy_description/meshes/Left.dae
- link r_wrist_abduction_link: geometry collision mesh filename=package://vizzy_description/meshes/M6R.dae; visual mesh filename=package://vizzy_description/meshes/M6R.dae
- link r_wrist_flection_link: geometry collision mesh filename=package://vizzy_description/meshes/M7R.dae; visual mesh filename=package://vizzy_description/meshes/M7R.dae
- link waist_link: geometry collision mesh filename=package://vizzy_description/meshes/M0.dae; visual mesh filename=package://vizzy_description/meshes/M0.dae

File: vizzy_description/robots/vizzy-no-collisions.urdf.xacro (robot description, xacro)
@@ -1,7 +1,7 @@
 <robot
-  name="vizzy-description"
+  name="vizzy_description"
   xmlns:xacro="http://ros.org/wiki/xacro" >
-  <xacro:include filename="$(find vizzy-description)/urdf/common.urdf.xacro" />
-  <xacro:include filename="$(find vizzy-description)/urdf/mounts/hokuyo_mount.urdf.xacro" />
+  <xacro:include filename="$(find vizzy_description)/urdf/common.urdf.xacro" />
+  <xacro:include filename="$(find vizzy_description)/urdf/mounts/hokuyo_mount.urdf.xacro" />
   <!-- root link, on the ground just below the robot origin -->
     <link name="base_footprint">
@@ -40,5 +40,5 @@
       <geometry>
         <mesh
-          filename="package://vizzy-description/meshes/Segway.dae" />
+          filename="package://vizzy_description/meshes/Segway.dae" />
       </geometry>
       <material
@@ -54,5 +54,5 @@
       <geometry>
         <mesh
-          filename="package://vizzy-description/meshes/Segway.dae" />
+          filename="package://vizzy_description/meshes/Segway.dae" />
       </geometry>
     </collision>
@@ -80,5 +80,5 @@
       <geometry>
         <mesh
-          filename="package://vizzy-description/meshes/Front.dae" />
+          filename="package://vizzy_description/meshes/Front.dae" />
       </geometry>
       <material
@@ -94,5 +94,5 @@
       <geometry>
         <mesh
-          filename="package://vizzy-description/meshes/Front.dae" />
+          filename="package://vizzy_description/meshes/Front.dae" />
       </geometry>
     </collision>
@@ -133,5 +133,5 @@
       <geometry>
         <mesh
-          filename="package://vizzy-description/meshes/F_W.dae" />
+          filename="package://vizzy_description/meshes/F_W.dae" />
       </geometry>
       <material
@@ -147,5 +147,5 @@
       <geometry>
         <mesh
-          filename="package://vizzy-description/meshes/F_W.dae" />
+          filename="package://vizzy_description/meshes/F_W.dae" />
       </geometry>
     </collision>
@@ -186,5 +186,5 @@
       <geometry>
         <mesh
-          filename="package://vizzy-description/meshes/Back.dae" />
+          filename="package://vizzy_description/meshes/Back.dae" />
       </geometry>
       <material
@@ -200,5 +200,5 @@
       <geometry>
         <mesh
-          filename="package://vizzy-description/meshes/Back.dae" />
+          filename="package://vizzy_description/meshes/Back.dae" />
       </geometry>
     </collision>
@@ -239,5 +239,5 @@
       <geometry>
         <mesh
-          filename="package://vizzy-description/meshes/B_W.dae" />
+          filename="package://vizzy_description/meshes/B_W.dae" />
       </geometry>
       <material
@@ -253,5 +253,5 @@
       <geometry>
         <mesh
-          filename="package://vizzy-description/meshes/B_W.dae" />
+          filename="package://vizzy_description/meshes/B_W.dae" />
       </geometry>
     </collision>
@@ -292,5 +292,5 @@
       <geometry>
         <mesh
-          filename="package://vizzy-description/meshes/Left.dae" />
+          filename="package://vizzy_description/meshes/Left.dae" />
       </geometry>
       <material
@@ -306,5 +306,5 @@
       <geometry>
         <mesh
-          filename="package://vizzy-description/meshes/Left.dae" />
+          filename="package://vizzy_description/meshes/Left.dae" />
       </geometry>
     </collision>
@@ -345,5 +345,5 @@
       <geometry>
         <mesh
-          filename="package://vizzy-description/meshes/Right.dae" />
+          filename="package://vizzy_description/meshes/Right.dae" />
       </geometry>
       <material
@@ -359,5 +359,5 @@
       <geometry>
         <mesh
-          filename="package://vizzy-description/meshes/Right.dae" />
+          filename="package://vizzy_description/meshes/Right.dae" />
       </geometry>
     </collision>
@@ -398,5 +398,5 @@
       <geometry>
         <mesh
-          filename="package://vizzy-description/meshes/M0.dae" />
+          filename="package://vizzy_description/meshes/M0.dae" />
       </geometry>
       <material
@@ -443,5 +443,5 @@
       <geometry>
         <mesh
-          filename="package://vizzy-description/meshes/M0L.dae" />
+          filename="package://vizzy_description/meshes/M0L.dae" />
       </geometry>
       <material
@@ -488,5 +488,5 @@
       <geometry>
         <mesh
-          filename="package://vizzy-description/meshes/M1L.dae" />
+          filename="package://vizzy_description/meshes/M1L.dae" />
       </geometry>
       <material
@@ -533,5 +533,5 @@
       <geometry>
         <mesh
-          filename="package://vizzy-description/meshes/M2L.dae" />
+          filename="package://vizzy_description/meshes/M2L.dae" />
       </geometry>
       <material
@@ -578,5 +578,5 @@
       <geometry>
         <mesh
-          filename="package://vizzy-description/meshes/M3L.dae" />
+          filename="package://vizzy_description/meshes/M3L.dae" />
       </geometry>
       <material
@@ -623,5 +623,5 @@
       <geometry>
         <mesh
-          filename="package://vizzy-description/meshes/M4L.dae" />
+          filename="package://vizzy_description/meshes/M4L.dae" />
       </geometry>
       <material
@@ -668,5 +668,5 @@
       <geometry>
         <mesh
-          filename="package://vizzy-description/meshes/M5L.dae" />
+          filename="package://vizzy_description/meshes/M5L.dae" />
       </geometry>
       <material
@@ -713,5 +713,5 @@
       <geometry>
         <mesh
-          filename="package://vizzy-description/meshes/M6L.dae" />
+          filename="package://vizzy_description/meshes/M6L.dae" />
       </geometry>
       <material
@@ -758,5 +758,5 @@
       <geometry>
         <mesh
-          filename="package://vizzy-description/meshes/M7L.dae" />
+          filename="package://vizzy_description/meshes/M7L.dae" />
       </geometry>
       <material
@@ -816,5 +816,5 @@
       <geometry>
         <mesh
-          filename="package://vizzy-description/meshes/M0R.dae" />
+          filename="package://vizzy_description/meshes/M0R.dae" />
       </geometry>
       <material
@@ -861,5 +861,5 @@
       <geometry>
         <mesh
-          filename="package://vizzy-description/meshes/M1R.dae" />
+          filename="package://vizzy_description/meshes/M1R.dae" />
       </geometry>
       <material
@@ -906,5 +906,5 @@
       <geometry>
         <mesh
-          filename="package://vizzy-description/meshes/M2R.dae" />
+          filename="package://vizzy_description/meshes/M2R.dae" />
       </geometry>
       <material
@@ -951,5 +951,5 @@
       <geometry>
         <mesh
-          filename="package://vizzy-description/meshes/M3R.dae" />
+          filename="package://vizzy_description/meshes/M3R.dae" />
       </geometry>
       <material
@@ -996,5 +996,5 @@
       <geometry>
         <mesh
-          filename="package://vizzy-description/meshes/M4R.dae" />
+          filename="package://vizzy_description/meshes/M4R.dae" />
       </geometry>
       <material
@@ -1041,5 +1041,5 @@
       <geometry>
         <mesh
-          filename="package://vizzy-description/meshes/M5R.dae" />
+          filename="package://vizzy_description/meshes/M5R.dae" />
       </geometry>
       <material
@@ -1086,5 +1086,5 @@
       <geometry>
         <mesh
-          filename="package://vizzy-description/meshes/M6R.dae" />
+          filename="package://vizzy_description/meshes/M6R.dae" />
       </geometry>
       <material
@@ -1131,5 +1131,5 @@
       <geometry>
         <mesh
-          filename="package://vizzy-description/meshes/M7R.dae" />
+          filename="package://vizzy_description/meshes/M7R.dae" />
       </geometry>
       <material
@@ -1189,5 +1189,5 @@
       <geometry>
         <mesh
-          filename="package://vizzy-description/meshes/M1.dae" />
+          filename="package://vizzy_description/meshes/M1.dae" />
       </geometry>
       <material
@@ -1234,5 +1234,5 @@
       <geometry>
         <mesh
-          filename="package://vizzy-description/meshes/M2.dae" />
+          filename="package://vizzy_description/meshes/M2.dae" />
       </geometry>
       <material
@@ -1279,5 +1279,5 @@
       <geometry>
         <mesh
-          filename="package://vizzy-description/meshes/M3.dae" />
+          filename="package://vizzy_description/meshes/M3.dae" />
       </geometry>
       <material
@@ -1324,5 +1324,5 @@
       <geometry>
         <mesh
-          filename="package://vizzy-description/meshes/M4.dae" />
+          filename="package://vizzy_description/meshes/M4.dae" />
       </geometry>
       <material
@@ -1382,5 +1382,5 @@
       <geometry>
         <mesh
-          filename="package://vizzy-description/meshes/M4.dae" />
+          filename="package://vizzy_description/meshes/M4.dae" />
       </geometry>
       <material

File: vizzy_description/robots/vizzy-with-collisions.urdf.xacro (robot description, xacro)
@@ -3,16 +3,16 @@
   <!-- The following included files set up definitions of parts of the robot body -->
   <!-- misc common stuff -->
-  <xacro:include filename="$(find vizzy-description)/urdf/common.urdf.xacro" />
-  <xacro:include filename="$(find vizzy-description)/urdf/mounts/hokuyo_mount.urdf.xacro" />
+  <xacro:include filename="$(find vizzy_description)/urdf/common.urdf.xacro" />
+  <xacro:include filename="$(find vizzy_description)/urdf/mounts/hokuyo_mount.urdf.xacro" />
   <!-- Vizzy base -->
-  <xacro:include filename="$(find vizzy-description)/urdf/base/base.urdf.xacro" />
+  <xacro:include filename="$(find vizzy_description)/urdf/base/base.urdf.xacro" />
   <!-- Vizzy torso -->
-  <xacro:include filename="$(find vizzy-description)/urdf/torso/torso.urdf.xacro" />
+  <xacro:include filename="$(find vizzy_description)/urdf/torso/torso.urdf.xacro" />
   <!-- Vizzy head -->
-  <xacro:include filename="$(find vizzy-description)/urdf/head/head.urdf.xacro" />
+  <xacro:include filename="$(find vizzy_description)/urdf/head/head.urdf.xacro" />
   <!-- Vizzy left arm -->
-  <xacro:include filename="$(find vizzy-description)/urdf/arm/left_arm.urdf.xacro" />
+  <xacro:include filename="$(find vizzy_description)/urdf/arm/left_arm.urdf.xacro" />
   <!-- Vizzy right arm -->
-  <xacro:include filename="$(find vizzy-description)/urdf/arm/right_arm.urdf.xacro" />
+  <xacro:include filename="$(find vizzy_description)/urdf/arm/right_arm.urdf.xacro" />
   <xacro:base name="base"/>
   <xacro:torso name="torso"/>
