Commit message: finished adding transmissions

File: vizzy_description/robots/vizzy.urdf.xacro (robot description, xacro)
@@ -32,11 +32,11 @@
   <xacro:head name="head"/>
   <!-- instantiate left arm -->
-  <xacro:leftarm name="left_arm" parent="M0" sufix="l" reflect="1">
+  <xacro:left_arm name="left_arm" parent="M0" sufix="l" reflect="1">
     <origin xyz="-0.01707 0.0 0.38145" rpy="0.0 0.0 0.0" />
-  </xacro:leftarm>
+  </xacro:left_arm>
   <!-- instantiate right arm -->
-  <xacro:rightarm name="right_arm" parent="M0" sufix="r" reflect="1">
+  <xacro:right_arm name="right_arm" parent="M0" sufix="r" reflect="1">
     <origin xyz="-0.01707 0.0 0.38145" rpy="0.0 0.0 0.0" />
-  </xacro:rightarm>
+  </xacro:right_arm>
   <!-- instantiate hokuyo -->
   <xacro:hokuyo_mount name="nav_hokuyo" parent="base" length="${SENSOR_BEAM_LENGTH*INCH_TO_M}" ros_topic="scan" update_rate="10" min_angle="${-(5 * M_PI)/12}" max_angle="${(5 * M_PI)/12}">

File: vizzy_description/urdf/arm/left_arm.gazebo.xacro (robot description, xacro)
@@ -1,3 +1,41 @@
 <?xml version="1.0"?>
 <robot xmlns:xacro="http://ros.org/wiki/xacro">
+  <xacro:macro name="left_arm_gazebo">
+    <gazebo reference="l_shoulder_scapula_link">
+      <mu1>0.2</mu1>
+      <mu2>0.2</mu2>
+    </gazebo>
+    <gazebo reference="l_shoulder_flection_link">
+      <mu1>0.2</mu1>
+      <mu2>0.2</mu2>
+    </gazebo>
+    <gazebo reference="l_shoulder_abduction_link">
+      <mu1>0.2</mu1>
+      <mu2>0.2</mu2>
+    </gazebo>
+    <gazebo reference="l_shoulder_rotation_link">
+      <mu1>0.2</mu1>
+      <mu2>0.2</mu2>
+    </gazebo>
+    <gazebo reference="l_elbow_flection_link">
+      <mu1>0.2</mu1>
+      <mu2>0.2</mu2>
+    </gazebo>
+    <gazebo reference="l_forearm_pronation_link">
+      <mu1>0.2</mu1>
+      <mu2>0.2</mu2>
+    </gazebo>
+    <gazebo reference="l_wrist_abduction_link">
+      <mu1>0.2</mu1>
+      <mu2>0.2</mu2>
+    </gazebo>
+    <gazebo reference="l_wrist_flection_link">
+      <mu1>0.2</mu1>
+      <mu2>0.2</mu2>
+    </gazebo>
+    <gazebo reference="l_palm_link">
+      <mu1>0.2</mu1>
+      <mu2>0.2</mu2>
+    </gazebo>
+  </xacro:macro>
 </robot>

File: vizzy_description/urdf/arm/left_arm.urdf.xacro (robot description, xacro)
@@ -4,451 +4,456 @@
        xmlns:interface="http://playerstage.sourceforge.net/gazebo/xmlschema/#interface"
        xmlns:xacro="http://ros.org/wiki/xacro">
- <xacro:macro name="leftarm" params="name parent sufix reflect *origin">
-  <link name="l_shoulder_scapula_link">
-    <inertial>
-      <origin
-        xyz="0.0 0.0 -0.16"
-        rpy="0.0 0.0 0.0" />
-      <mass
-        value="0.328838093974495" />
-      <inertia
-        ixx="0.00123108428695023"
-        ixy="-7.89159441144304E-11"
-        ixz="6.34904994947113E-10"
-        iyy="0.000919898935947314"
-        iyz="7.50425183645029E-05"
-        izz="0.000480033534091429" />
-    </inertial>
-    <visual>
-      <origin
-        xyz="0.0 0.0 -0.16"
-        rpy="0.0 0.0 0.0" />
-      <geometry>
-        <mesh
-          filename="package://vizzy_description/meshes/M0L.dae" />
-      </geometry>
-      <material
-        name="">
-        <color
-          rgba="0.898039215686275 0.917647058823529 0.929411764705882 1" />
-      </material>
-    </visual>
-    <collision>
-      <origin
-        xyz="0.0 0.0 -0.16"
-        rpy="0.0 0.0 0.0" />
-      <geometry>
-        <mesh
-          filename="package://vizzy_description/meshes/M0L.dae" />
-      </geometry>
-    </collision>
-  </link>
-  <joint
-    name="l_shoulder_scapula_joint"
-    type="revolute">
-    <origin
-      xyz="0.0 0.0 0.0805"
-      rpy="${M_PI/2.0} 0.0 0.0" />
-    <parent
-      link="waist_link" />
-    <child
-      link="l_shoulder_scapula_link" />
-    <axis
-      xyz="0 0 1" />
-    <limit lower="-0.314159265" upper="0.314159265" effort="10" velocity="3" />
-  </joint>
-  <link
-    name="l_shoulder_flection_link">
-    <inertial>
-      <origin
-        xyz="0.0 0.0 -0.0479999999999997"
-        rpy="0.0 0.0 -4.1963" />
-      <mass
-        value="0.329707501986262" />
-      <inertia
-        ixx="0.00116793344879787"
-        ixy="0.000134890277431864"
-        ixz="-3.78918978637635E-05"
-        iyy="0.0010123206932222"
-        iyz="-6.56607930808342E-05"
-        izz="0.000480378945367471" />
-    </inertial>
-    <visual>
-      <origin
-        xyz="0.0 0.0 -0.0479999999999997"
-        rpy="0.0 0.0 -4.1963" />
-      <geometry>
-        <mesh
-          filename="package://vizzy_description/meshes/M1L.dae" />
-      </geometry>
-      <material
-        name="">
-        <color
-          rgba="0.898039215686275 0.917647058823529 0.929411764705882 1" />
-      </material>
-    </visual>
-    <collision>
-      <origin
-        xyz="0.0 0.0 -0.0479999999999997"
-        rpy="0.0 0.0 -4.1963" />
-      <geometry>
-        <mesh
-          filename="package://vizzy_description/meshes/M1L.dae" />
-      </geometry>
-    </collision>
-  </link>
-  <joint
-    name="l_shoulder_flection_joint"
-    type="revolute">
-    <origin
-      xyz="0.0 0.0 -0.212"
-      rpy="${M_PI/2.0} 0.0 0.0" />
-    <parent
-      link="l_shoulder_scapula_link" />
-    <child
-      link="l_shoulder_flection_link" />
-    <axis
-      xyz="0 0 1" />
-    <limit lower="-1.30899694" upper="2.35619449" effort="10" velocity="3" />
-  </joint>
-  <link
-    name="l_shoulder_abduction_link">
-    <inertial>
-      <origin
-        xyz="-0.034 -0.009 -0.001"
-        rpy="0.0 0.0 -4.3633" />
-      <mass
-        value="0.337952134412867" />
-      <inertia
-        ixx="0.000722844157573501"
-        ixy="4.62401523525089E-05"
-        ixz="1.45397456168781E-06"
-        iyy="0.000316566987264746"
-        iyz="1.40155768711965E-05"
-        izz="0.000577759873964217" />
-    </inertial>
-    <visual>
-      <origin
-        xyz="-0.034 -0.009 -0.001"
-        rpy="0.0 0.0 -4.3633" />
-      <geometry>
-        <mesh
-          filename="package://vizzy_description/meshes/M2L.dae" />
-      </geometry>
-      <material
-        name="">
-        <color
-          rgba="0.898039215686275 0.917647058823529 0.929411764705882 1" />
-      </material>
-    </visual>
-    <collision>
-      <origin
-        xyz="-0.034 -0.009 -0.001"
-        rpy="0.0 0.0 -4.3633" />
-      <geometry>
-        <mesh
-          filename="package://vizzy_description/meshes/M2L.dae" />
-      </geometry>
-    </collision>
-  </link>
-  <joint
-    name="l_shoulder_abduction_joint"
-    type="revolute">
-    <origin
-      xyz="0.0 0.0 -0.10256"
-      rpy="${M_PI/2.0} 0.0 ${-M_PI/2.0}" />
-    <parent
-      link="l_shoulder_flection_link" />
-    <child
-      link="l_shoulder_abduction_link" />
-    <axis
-      xyz="0 0 1" />
-    <limit lower="0" upper="1.30899694" effort="10" velocity="3" />
-  </joint>
-  <link
-    name="l_shoulder_rotation_link">
-    <inertial>
-      <origin
-        xyz="0.003 -0.006 -0.127"
-        rpy="0.0 0.0 ${M_PI/2}" />
-      <mass
-        value="0.302328099651438" />
-      <inertia
-        ixx="0.00061524641225989"
-        ixy="4.12484077822449E-06"
-        ixz="6.13276820445825E-05"
-        iyy="0.000574848729857274"
-        iyz="-2.49114687077784E-05"
-        izz="0.000240227009768201" />
-    </inertial>
-    <visual>
-      <origin
-        xyz="0.003 -0.006 -0.127"
-        rpy="0.0 0.0 ${M_PI/2}" />
-      <geometry>
-        <mesh
-          filename="package://vizzy_description/meshes/M3L.dae" />
-      </geometry>
-      <material
-        name="">
-        <color
-          rgba="0.898039215686275 0.917647058823529 0.929411764705882 1" />
-      </material>
-    </visual>
-    <collision>
-      <origin
-        xyz="0.003 -0.006 -0.127"
-        rpy="0.0 0.0 ${M_PI/2}" />
-      <geometry>
-        <mesh
-          filename="package://vizzy_description/meshes/M3L.dae" />
-      </geometry>
-    </collision>
-  </link>
-  <joint
-    name="l_shoulder_rotation_joint"
-    type="revolute">
-    <origin
-      xyz="0.0 0.0 0.0"
-      rpy="${M_PI/2.0} 0.0 ${11*M_PI/18}" />
-    <parent
-      link="l_shoulder_abduction_link" />
-    <child
-      link="l_shoulder_rotation_link" />
-    <axis
-      xyz="0 0 1" />
-    <limit lower="-1.48352986" upper="1.48352986" effort="10" velocity="3" />
-  </joint>
-  <link
-    name="l_elbow_flection_link">
-    <inertial>
-      <origin
-        xyz="0.002 -0.035 0.0"
-        rpy="0.0 ${M_PI} ${M_PI}" />
-      <mass
-        value="0.224019872188573" />
-      <inertia
-        ixx="0.000224266883987209"
-        ixy="-7.91977708288826E-06"
-        ixz="-2.45971183993369E-07"
-        iyy="9.89759646705347E-05"
-        iyz="9.59757272005961E-06"
-        izz="0.000213841891548227" />
-    </inertial>
-    <visual>
-      <origin
-        xyz="0.002 -0.035 0.0"
-        rpy="0.0 ${M_PI} ${M_PI}" />
-      <geometry>
-        <mesh
-          filename="package://vizzy_description/meshes/M4L.dae" />
-      </geometry>
-      <material
-        name="">
-        <color
-          rgba="0.898039215686275 0.917647058823529 0.929411764705882 1" />
-      </material>
-    </visual>
-    <collision>
-      <origin
-        xyz="0.002 -0.035 0.0"
-        rpy="0.0 ${M_PI} ${M_PI}" />
-      <geometry>
-        <mesh
-          filename="package://vizzy_description/meshes/M4L.dae" />
-      </geometry>
-    </collision>
-  </link>
-  <joint
-    name="l_elbow_flection_joint"
-    type="revolute">
-    <origin
-      xyz="0.0 0.0 -0.16296"
-      rpy="${M_PI/2.0} 0.0 ${M_PI/2.0} " />
-    <parent
-      link="l_shoulder_rotation_link" />
-    <child
-      link="l_elbow_flection_link" />
-    <axis
-      xyz="0 0 1" />
-    <limit lower="0" upper="1.91986218" effort="10" velocity="3" />
-  </joint>
-  <link
-    name="l_forearm_pronation_link">
-    <inertial>
-      <origin
-        xyz="0.000 0.007 0.11"
-        rpy="0.0 ${M_PI} ${-M_PI/2}" />
-      <mass
-        value="0.192525480880953" />
-      <inertia
-        ixx="0.000215803121531384"
-        ixy="6.01824209118801E-08"
-        ixz="-9.78525879865635E-06"
-        iyy="0.000229047941469006"
-        iyz="-3.21836442544262E-07"
-        izz="0.000102658857339667" />
-    </inertial>
-    <visual>
-      <origin
-        xyz="0.000 0.007 0.11"
-        rpy="0.0 ${M_PI} ${-M_PI/2}" />
-      <geometry>
-        <mesh
-          filename="package://vizzy_description/meshes/M5L.dae" />
-      </geometry>
-      <material
-        name="">
-        <color
-          rgba="0.898039215686275 0.917647058823529 0.929411764705882 1" />
-      </material>
-    </visual>
-    <collision>
-      <origin
-        xyz="0.000 0.007 0.11"
-        rpy="0.0 ${M_PI} ${-M_PI/2}" />
-      <geometry>
-        <mesh
-          filename="package://vizzy_description/meshes/M5L.dae" />
-      </geometry>
-    </collision>
-  </link>
-  <joint
-    name="l_forearm_pronation_joint"
-    type="revolute">
-    <origin
-      xyz="0.0 0.0 0.0"
-      rpy="${M_PI/2} 0.0 0.0" />
-    <parent
-      link="l_elbow_flection_link" />
-    <child
-      link="l_forearm_pronation_link" />
-    <axis
-      xyz="0 0 1" />
-    <limit lower="-1.48352986" upper="1.48352986" effort="10" velocity="3" />
-  </joint>
-  <link
-    name="l_wrist_abduction_link">
-    <inertial>
-      <origin
-        xyz="-0.0047 -0.022 0.003"
-        rpy="${M_PI/2} 0.0 ${-M_PI/4}" />
-      <mass
-        value="0.151302636921624" />
-      <inertia
-        ixx="0.000116373512947626"
-        ixy="1.31009871908069E-05"
-        ixz="6.69703789973942E-05"
-        iyy="0.00020031628400595"
-        iyz="1.00268924727662E-05"
-        izz="0.000162164313365602" />
-    </inertial>
-    <visual>
-      <origin
-        xyz="-0.0047 -0.020 0.003"
-        rpy="${M_PI/2} 0.0 ${-M_PI/4}" />
-      <geometry>
-        <mesh
-          filename="package://vizzy_description/meshes/M6L.dae" />
-      </geometry>
-      <material
-        name="">
-        <color
-          rgba="0.898039215686275 0.917647058823529 0.929411764705882 1" />
-      </material>
-    </visual>
-    <collision>
-      <origin
-        xyz="-0.0047 -0.022 0.003"
-        rpy="${M_PI/2} 0.0 ${-M_PI/4}" />
-      <geometry>
-        <mesh
-          filename="package://vizzy_description/meshes/M6L.dae" />
-      </geometry>
-    </collision>
-  </link>
-  <joint
-    name="l_wrist_abduction_joint"
-    type="revolute">
-    <origin
-      xyz="0.0 0.0 0.18925"
-      rpy="${M_PI/2.0} 0.0 0.0" />
-    <parent
-      link="l_forearm_pronation_link" />
-    <child
-      link="l_wrist_abduction_link" />
-    <axis
-      xyz="0 0 1" />
-    <limit lower="-0.610865238" upper="0.610865238" effort="10" velocity="3" />
-  </joint>
-  <link
-    name="l_wrist_flection_link">
-    <inertial>
-      <origin
-        xyz="-0.106 -0.0077 -0.015"
-        rpy="0.0 0.0 ${M_PI/2.0}" />
-      <mass
-        value="0.263177712190575" />
-      <inertia
-        ixx="0.00141536691437145"
-        ixy="-5.47006881402205E-06"
-        ixz="4.93141952833896E-05"
-        iyy="0.000423837541639676"
-        iyz="0.000132116163317958"
-        izz="0.0010337584021873" />
-    </inertial>
-    <visual>
-      <origin
-        xyz="-0.106 -0.0077 -0.015"
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
File: vizzy_description/urdf/arm/right_arm.gazebo.xacro (robot description, xacro)
@@ -1,3 +1,41 @@
 <?xml version="1.0"?>
 <robot xmlns:xacro="http://ros.org/wiki/xacro">
+  <xacro:macro name="right_arm_gazebo">
+    <gazebo reference="r_shoulder_scapula_link">
+      <mu1>0.2</mu1>
+      <mu2>0.2</mu2>
+    </gazebo>
+    <gazebo reference="r_shoulder_flection_link">
+      <mu1>0.2</mu1>
+      <mu2>0.2</mu2>
+    </gazebo>
+    <gazebo reference="r_shoulder_abduction_link">
+      <mu1>0.2</mu1>
+      <mu2>0.2</mu2>
+    </gazebo>
+    <gazebo reference="r_shoulder_rotation_link">
+      <mu1>0.2</mu1>
+      <mu2>0.2</mu2>
+    </gazebo>
+    <gazebo reference="r_elbow_flection_link">
+      <mu1>0.2</mu1>
+      <mu2>0.2</mu2>
+    </gazebo>
+    <gazebo reference="r_forearm_pronation_link">
+      <mu1>0.2</mu1>
+      <mu2>0.2</mu2>
+    </gazebo>
+    <gazebo reference="r_wrist_abduction_link">
+      <mu1>0.2</mu1>
+      <mu2>0.2</mu2>
+    </gazebo>
+    <gazebo reference="r_wrist_flection_link">
+      <mu1>0.2</mu1>
+      <mu2>0.2</mu2>
+    </gazebo>
+    <gazebo reference="r_palm_link">
+      <mu1>0.2</mu1>
+      <mu2>0.2</mu2>
+    </gazebo>
+  </xacro:macro>
 </robot>
