Commit message: finished adding transmissions

File: vizzy_description/urdf/arm/right_arm.urdf.xacro (robot description, xacro)
@@ -4,451 +4,456 @@
        xmlns:interface="http://playerstage.sourceforge.net/gazebo/xmlschema/#interface"
        xmlns:xacro="http://ros.org/wiki/xacro">
- <xacro:macro name="rightarm" params="name parent sufix reflect *origin">
-  <link name="r_shoulder_scapula_link">
-    <inertial>
-      <origin
-        xyz="0 0 0.166"
-        rpy="0 ${-M_PI} ${M_PI}" />
-      <mass
-        value="0.328838093982794" />
-      <inertia
-        ixx="0.00123108428695986"
-        ixy="-7.89100940163704E-11"
-        ixz="6.34844936183615E-10"
-        iyy="0.000919898935949979"
-        iyz="7.50425183699034E-05"
-        izz="0.000480033534097503" />
-    </inertial>
-    <visual>
-      <origin
-        xyz="0 0 0.166"
-        rpy="0 ${-M_PI} ${M_PI}" />
-      <geometry>
-        <mesh
-          filename="package://vizzy_description/meshes/M0R.dae" />
-      </geometry>
-      <material
-        name="">
-        <color
-          rgba="0.898039215686275 0.917647058823529 0.929411764705882 1" />
-      </material>
-    </visual>
-    <collision>
-      <origin
-        xyz="0 0 0.166"
-        rpy="0 ${-M_PI} ${M_PI}" />
-      <geometry>
-        <mesh
-          filename="package://vizzy_description/meshes/M0R.dae" />
-      </geometry>
-    </collision>
-  </link>
-  <joint
-    name="r_shoulder_scapula_joint"
-    type="revolute">
-    <origin
-      xyz="0.0 0.0 -0.0805"
-      rpy="${M_PI/2.0} 0.0  ${M_PI}" />
-    <parent
-      link="waist_link" />
-    <child
-      link="r_shoulder_scapula_link" />
-    <axis
-      xyz="0 0 1" />
-    <limit lower="-0.314159265" upper="0.314159265" effort="10" velocity="3" />
-  </joint>
-  <link
-    name="r_shoulder_flection_link">
-    <inertial>
-      <origin
-        xyz="0.0 0.0 0.0479999999999997"
-        rpy="0.0 ${M_PI} -1.0547" />
-      <mass
-        value="0.32970750458976" />
-      <inertia
-        ixx="0.00116793345082586"
-        ixy="-0.000134890089770505"
-        ixz="3.78931445548874E-05"
-        iyy="0.00101232051019094"
-        iyz="-6.56607928268466E-05"
-        izz="0.000480378760663095" />
-    </inertial>
-    <visual>
-      <origin
-        xyz="0.0 0.0 0.0479999999999997"
-        rpy="0.0 ${M_PI} -1.0547" />
-      <geometry>
-        <mesh
-          filename="package://vizzy_description/meshes/M1R.dae" />
-      </geometry>
-      <material
-        name="">
-        <color
-          rgba="0.898039215686275 0.917647058823529 0.929411764705882 1" />
-      </material>
-    </visual>
-    <collision>
-      <origin
-        xyz="0.0 0.0 0.0479999999999997"
-        rpy="0.0 ${M_PI} -1.0547" />
-      <geometry>
-        <mesh
-          filename="package://vizzy_description/meshes/M1R.dae" />
-      </geometry>
-    </collision>
-  </link>
-  <joint
-    name="r_shoulder_flection_joint"
-    type="revolute">
-    <origin
-      xyz="0.0 0.0 0.212"
-      rpy="${M_PI/2.0} 0.0 0.0" />
-    <parent
-      link="r_shoulder_scapula_link" />
-    <child
-      link="r_shoulder_flection_link" />
-    <axis
-      xyz="0 0 1" />
-    <limit lower="-1.30899694" upper="2.35619449" effort="10" velocity="3" />
-  </joint>
-  <link
-    name="r_shoulder_abduction_link">
-    <inertial>
-      <origin
-        xyz="0.034 0.009 -0.001"
-        rpy="0 ${M_PI} -1.2217" />
-      <mass
-        value="0.337952134649786" />
-      <inertia
-        ixx="0.000722844158320218"
-        ixy="-4.62401500200836E-05"
-        ixz="-1.45396813798355E-06"
-        iyy="0.000316566986726189"
-        iyz="1.40155770580819E-05"
-        izz="0.00057775987279214" />
-    </inertial>
-    <visual>
-      <origin
-        xyz="0.034 0.009 -0.001"
-        rpy="0 ${M_PI} -1.2217" />
-      <geometry>
-        <mesh
-          filename="package://vizzy_description/meshes/M2R.dae" />
-      </geometry>
-      <material
-        name="">
-        <color
-          rgba="0.898039215686275 0.917647058823529 0.929411764705882 1" />
-      </material>
-    </visual>
-    <collision>
-      <origin
-        xyz="0.034 0.009 -0.001"
-        rpy="0 ${M_PI} -1.2217" />
-      <geometry>
-        <mesh
-          filename="package://vizzy_description/meshes/M2R.dae" />
-      </geometry>
-    </collision>
-  </link>
-  <joint
-    name="r_shoulder_abduction_joint"
-    type="revolute">
-    <origin
-      xyz="0.0 0.0 0.10256"
-      rpy="${M_PI/2.0} 0.0 ${-M_PI/2.0}" />
-    <parent
-      link="r_shoulder_flection_link" />
-    <child
-      link="r_shoulder_abduction_link" />
-    <axis
-      xyz="0 0 1" />
-    <limit lower="0" upper="1.30899694" effort="10" velocity="3" />
-  </joint>
-  <link
-    name="r_shoulder_rotation_link">
-    <inertial>
-      <origin
-        xyz="-0.003 0.006 0.127"
-        rpy="${M_PI} 0 ${M_PI/2}" />
-      <mass
-        value="0.302328098083101" />
-      <inertia
-        ixx="0.000615246412768918"
-        ixy="-4.12473635541355E-06"
-        ixz="-6.13280078197927E-05"
-        iyy="0.000574849538917934"
-        iyz="-2.49114717380023E-05"
-        izz="0.000240227819685505" />
-    </inertial>
-    <visual>
-      <origin
-        xyz="-0.003 0.006 0.127"
-        rpy="${M_PI} 0 ${M_PI/2}" />
-      <geometry>
-        <mesh
-          filename="package://vizzy_description/meshes/M3R.dae" />
-      </geometry>
-      <material
-        name="">
-        <color
-          rgba="0.898039215686275 0.917647058823529 0.929411764705882 1" />
-      </material>
-    </visual>
-    <collision>
-      <origin
-        xyz="-0.003 0.006 0.127"
-        rpy="${M_PI} 0 ${M_PI/2}" />
-      <geometry>
-        <mesh
-          filename="package://vizzy_description/meshes/M3R.dae" />
-      </geometry>
-    </collision>
-  </link>
-  <joint
-    name="r_shoulder_rotation_joint"
-    type="revolute">
-    <origin
-      xyz="0.0 0.0 0.0"
-      rpy="${M_PI/2.0} 0.0 ${11*M_PI/18}" />
-    <parent
-      link="r_shoulder_abduction_link" />
-    <child
-      link="r_shoulder_rotation_link" />
-    <axis
-      xyz="0 0 1" />
-    <limit lower="-1.48352986" upper="1.48352986" effort="10" velocity="3" />
-  </joint>
-  <link
-    name="r_elbow_flection_link">
-    <inertial>
-      <origin
-        xyz="-0.002 0.035 0.0"
-        rpy="0.0 0.0 0.0" />
-      <mass
-        value="0.224019872068973" />
-      <inertia
-        ixx="0.000224266812490421"
-        ixy="7.91977782063514E-06"
-        ixz="2.45606472556753E-07"
-        iyy="9.89758932648508E-05"
-        iyz="9.59616898464483E-06"
-        izz="0.000213841891572994" />
-    </inertial>
-    <visual>
-      <origin
-        xyz="-0.002 0.035 0.0"
-        rpy="0.0 0.0 0.0" />
-      <geometry>
-        <mesh
-          filename="package://vizzy_description/meshes/M4R.dae" />
-      </geometry>
-      <material
-        name="">
-        <color
-          rgba="0.898039215686275 0.917647058823529 0.929411764705882 1" />
-      </material>
-    </visual>
-    <collision>
-      <origin
-        xyz="-0.002 0.035 0.0"
-        rpy="0.0 0.0 0.0" />
-      <geometry>
-        <mesh
-          filename="package://vizzy_description/meshes/M4R.dae" />
-      </geometry>
-    </collision>
-  </link>
-  <joint
-    name="r_elbow_flection_joint"
-    type="revolute">
-    <origin
-      xyz="0.0 0.0 0.16296"
-      rpy="${M_PI/2.0} 0.0 ${M_PI/2.0}" />
-    <parent
-      link="r_shoulder_rotation_link" />
-    <child
-      link="r_elbow_flection_link" />
-    <axis
-      xyz="0 0 1" />
-    <limit lower="0" upper="1.91986218" effort="10" velocity="3" />
-  </joint>
-  <link
-    name="r_forearm_pronation_link">
-    <inertial>
-      <origin
-        xyz="0.00 -0.007 -0.11"
-        rpy="0.0 0.0 ${M_PI/2}" />
-      <mass
-        value="0.19252548105039" />
-      <inertia
-        ixx="0.000215803119910502"
-        ixy="-6.086463167521E-08"
-        ixz="9.78455040630467E-06"
-        iyy="0.000229047404557263"
-        iyz="-3.19642916101682E-07"
-        izz="0.000102658318305363" />
-    </inertial>
-    <visual>
-      <origin
-        xyz="0.00 -0.007 -0.11"
-        rpy="0.0 0.0 ${M_PI/2}" />
-      <geometry>
-        <mesh
-          filename="package://vizzy_description/meshes/M5R.dae" />
-      </geometry>
-      <material
-        name="">
-        <color
-          rgba="0.898039215686275 0.917647058823529 0.929411764705882 1" />
-      </material>
-    </visual>
-    <collision>
-      <origin
-        xyz="0.00 -0.007 -0.11"
-        rpy="0.0 0.0 ${M_PI/2}" />
-      <geometry>
-        <mesh
-          filename="package://vizzy_description/meshes/M5R.dae" />
-      </geometry>
-    </collision>
-  </link>
-  <joint
-    name="r_forearm_pronation_joint"
-    type="revolute">
-    <origin
-      xyz="0.0 0.0 0.0"
-      rpy="${M_PI/2.0} 0.0 0.0" />
-    <parent
-      link="r_elbow_flection_link" />
-    <child
-      link="r_forearm_pronation_link" />
-    <axis
-      xyz="0 0 1" />
-    <limit lower="-1.48352986" upper="1.48352986" effort="10" velocity="3" />
-  </joint>
-  <link
-    name="r_wrist_abduction_link">
-    <inertial>
-      <origin
-        xyz="0.0047 0.028 -0.003"
-        rpy="${M_PI} ${M_PI} 0" />
-      <mass
-        value="0.15130263687109" />
-      <inertia
-        ixx="0.000206280948481805"
-        ixy="-2.10167871847464E-05"
-        ixz="-1.95502541303483E-06"
-        iyy="7.18084114032176E-05"
-        iyz="1.63557763545568E-05"
-        izz="0.000199867817507994" />
-    </inertial>
-    <visual>
-      <origin
-        xyz="0.0047 0.028 -0.003"
-        rpy="${M_PI} ${M_PI} 0" />
-      <geometry>
-        <mesh
-          filename="package://vizzy_description/meshes/M6R.dae" />
-      </geometry>
-      <material
-        name="">
-        <color
-          rgba="0.898039215686275 0.917647058823529 0.929411764705882 1" />
-      </material>
-    </visual>
-    <collision>
-      <origin
-        xyz="0.0047 0.028 -0.003"
-        rpy="${M_PI} ${M_PI} 0" />
-      <geometry>
-        <mesh
-          filename="package://vizzy_description/meshes/M6R.dae" />
-      </geometry>
-    </collision>
-  </link>
-  <joint
-    name="r_wrist_abduction_joint"
-    type="revolute">
-    <origin
-      xyz="0.0 0.0 -0.18925"
-      rpy="${M_PI/2.0} 0.0 0.0" />
-    <parent
-      link="r_forearm_pronation_link" />
-    <child
-      link="r_wrist_abduction_link" />
-    <axis
-      xyz="0 0 1" />
-    <limit lower="-0.610865238" upper="0.610865238" effort="10" velocity="3" />
-  </joint>
-  <link
-    name="r_wrist_flection_link">
-    <inertial>
-      <origin
-        xyz="0.106 0.0077 0.017"
-        rpy="0.0 ${M_PI} ${-M_PI/2}" />
-      <mass
-        value="0.263247942991542" />
-      <inertia
-        ixx="0.00142191847625323"
-        ixy="7.01996302951171E-06"
-        ixz="-4.24188980462336E-05"
-        iyy="0.000427941498537125"
-        iyz="0.000132013848915951"
-        izz="0.00103049250587026" />
-    </inertial>
-    <visual>
-      <origin
-        xyz="0.106 0.0077 0.017"
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
File: vizzy_description/urdf/base/base.gazebo.xacro (robot description, xacro)
@@ -30,18 +30,4 @@
       <stopKp value="1000.0" />
     </gazebo>-->
-    <gazebo>
-      <plugin name="differential_drive_controller" filename="libgazebo_ros_diff_drive.so">
-        <leftJoint>l_wheel_joint</leftJoint>
-        <rightJoint>r_wheel_joint</rightJoint>
-        <wheelSeparation>0.4580</wheelSeparation>
-        <wheelDiameter>0.2410</wheelDiameter>
-        <torque>20</torque>
-        <commandTopic>cmd_vel</commandTopic>
-        <odometryTopic>odom</odometryTopic>
-        <odometryFrame>odom</odometryFrame>
-        <robotBaseFrame>base_footprint</robotBaseFrame>
-        <updateRate>100.0</updateRate>
-      </plugin>
-    </gazebo>
   </xacro:macro>
 </robot>

File: vizzy_description/urdf/head/head.gazebo.xacro (robot description, xacro)
@@ -5,45 +5,20 @@
       <mu1>0.2</mu1>
       <mu2>0.2</mu2>
-      <turnGravityOff>true</turnGravityOff>
-    </gazebo>
-    <gazebo reference="neck_pan_joint">
-      <stopKd value="1.0" />
-      <stopKp value="1000000.0" />
     </gazebo>
     <gazebo reference="neck_tilt_link">
       <mu1>0.2</mu1>
       <mu2>0.2</mu2>
-      <kp value="1.0" />
-      <turnGravityOff>true</turnGravityOff>
-    </gazebo>
-    <gazebo reference="neck_tilt_joint">
-      <kd value="1000000.0" />
     </gazebo>
     <gazebo reference="eyes_tilt_link">
       <mu1>0.2</mu1>
       <mu2>0.2</mu2>
-      <turnGravityOff>true</turnGravityOff>
-    </gazebo>
-    <gazebo reference="eyes_tilt_joint">
-      <stopKd value="1.0" />
-      <stopKp value="1000000.0" />
     </gazebo>
     <gazebo reference="r_eye_pan_link">
       <mu1>0.2</mu1>
       <mu2>0.2</mu2>
-      <turnGravityOff>true</turnGravityOff>
-    </gazebo>
-    <gazebo reference="r_eye_pan_joint">
-      <stopKd value="1.0" />
-      <stopKp value="1000000.0" />
     </gazebo>
     <gazebo reference="l_eye_pan_link">
       <mu1>0.2</mu1>
       <mu2>0.2</mu2>
-      <turnGravityOff>true</turnGravityOff>
-    </gazebo>
-    <gazebo reference="l_eye_pan_joint">
-      <stopKd value="1.0" />
-      <stopKp value="1000000.0" />
     </gazebo>
   </xacro:macro>

File: vizzy_description/urdf/torso/torso.gazebo.xacro (robot description, xacro)
@@ -3,12 +3,7 @@
   <xacro:macro name="torso_gazebo">
     <gazebo reference="waist_link">
-      <gravity>false</gravity>
+      <mu1>0.2</mu1>
+      <mu2>0.2</mu2>
     </gazebo>
-    <!--<gazebo reference="waist_joint">
-      <kd>1.0</kd>
-      <kp>100000000.0</kp>
-      <stopKd value="1.0" />
-      <stopKp value="100000000.0" />
-    </gazebo>-->
   </xacro:macro>
 </robot>
