Commit message: changes in the eyes. Now we have vergence and version joints

File: vizzy_description/robots/vizzy.urdf.xacro (robot description, xacro)
@@ -28,11 +28,11 @@
   <xacro:head name="head"/>
   <!-- instantiate left arm -->
-  <xacro:left_arm name="left_arm" parent="waist_link" sufix="l" reflect="1">
+  <!--<xacro:left_arm name="left_arm" parent="waist_link" sufix="l" reflect="1">
     <origin xyz="-0.01707 0.0 0.38145" rpy="0.0 0.0 0.0" />
-  </xacro:left_arm>
+  </xacro:left_arm>-->
   <!-- instantiate right arm -->
-  <xacro:right_arm name="right_arm" parent="waist_link" sufix="r" reflect="1">
+  <!--<xacro:right_arm name="right_arm" parent="waist_link" sufix="r" reflect="1">
     <origin xyz="-0.01707 0.0 0.38145" rpy="0.0 0.0 0.0" />
-  </xacro:right_arm>
+  </xacro:right_arm>-->
   <!-- instantiate hokuyo -->
   <xacro:hokuyo_mount name="nav_hokuyo" parent="base" length="${SENSOR_BEAM_LENGTH*INCH_TO_M}" ros_topic="scan" update_rate="10" min_angle="${-(5 * M_PI)/12}" max_angle="${(5 * M_PI)/12}">

File: vizzy_description/urdf/head/head.gazebo.xacro (robot description, xacro)
@@ -5,21 +5,114 @@
       <mu1>0.2</mu1>
       <mu2>0.2</mu2>
+ 			<kp value="1000000.0" />
+			<kd value="1.0" />
     </gazebo>
     <gazebo reference="neck_tilt_link">
       <mu1>0.2</mu1>
       <mu2>0.2</mu2>
+ 			<kp value="1000000.0" />
+			<kd value="1.0" />
     </gazebo>
     <gazebo reference="eyes_tilt_link">
       <mu1>0.2</mu1>
       <mu2>0.2</mu2>
+ 			<kp value="1000000.0" />
+			<kd value="1.0" />
     </gazebo>
-    <gazebo reference="r_eye_pan_link">
+    <gazebo reference="version_link">
+    </gazebo>
+    <gazebo reference="r_eye_version_link">
+    </gazebo>
+    <gazebo reference="l_eye_version_link">
+    </gazebo>
+    <gazebo reference="vergence_link">
+      <gravity value="false"/>
       <mu1>0.2</mu1>
       <mu2>0.2</mu2>
+ 			<kp value="1000000.0" />
+			<kd value="1.0" />
     </gazebo>
-    <gazebo reference="l_eye_pan_link">
+		 <gazebo reference="r_eye_vergence_link">
       <mu1>0.2</mu1>
       <mu2>0.2</mu2>
+ 			<kp value="1000000.0" />
+			<kd value="1.0" />
     </gazebo>
+    <gazebo reference="l_eye_vergence_link">
+      <mu1>0.2</mu1>
+      <mu2>0.2</mu2>
+ 			<kp value="1000000.0" />
+			<kd value="1.0" />
+    </gazebo>
+ 		<gazebo reference="neck_pan_joint">
+			<kd value="1.0" />
+			<kp value="1000000.0" />
+			<fudgeFactor value="1.0" />
+			<provideFeedback value="true"/>
+		</gazebo>
+ 		<gazebo reference="neck_tilt_joint">
+			<kd value="1.0" />
+			<kp value="1000000.0" />
+			<fudgeFactor value="1.0" />
+			<provideFeedback value="true"/>
+		</gazebo>
+ 		<gazebo reference="eyes_tilt_joint">
+			<kd value="1.0" />
+			<kp value="1000000.0" />
+			<fudgeFactor value="1.0" />
+			<provideFeedback value="true"/>
+		</gazebo>
+ 		<gazebo reference="version_joint">
+  		<stopKd value="1000000.0" />
+  		<stopKp value="1000000.0" />
+		</gazebo>
+ 		<!--<gazebo reference="l_eye_version_joint">
+  		<stopKd value="1000000.0" />
+  		<stopKp value="1000000.0" />
+		</gazebo>
+ 		<gazebo reference="r_eye_version_joint">
+  		<stopKd value="1000000.0" />
+  		<stopKp value="1000000.0" />
+		</gazebo>-->
+ 		<gazebo reference="vergence_joint">
+  		<stopKd value="1000000.0" />
+  		<stopKp value="1000000.0" />
+		</gazebo>
+ 		<!--<gazebo reference="l_eye_vergence_joint">
+  		<stopKd value="1000000.0" />
+  		<stopKp value="1000000.0" />
+		</gazebo>
+ 		<gazebo reference="r_eye_vergence_joint">
+  		<stopKd value="1000000.0" />
+  		<stopKp value="1000000.0" />
+		</gazebo>-->
+		<gazebo>
+			<plugin name="mimic_plugin" filename="libgazebo_mimic_plugin.so">
+				<joint>version_joint</joint>
+				<mimicJoint>l_eye_version_joint</mimicJoint>
+				<multiplier>1.0</multiplier>
+			</plugin>
+		</gazebo>
+		<gazebo>
+			<plugin name="mimic_plugin" filename="libgazebo_mimic_plugin.so">
+				<joint>version_joint</joint>
+				<mimicJoint>r_eye_version_joint</mimicJoint>
+				<multiplier>1.0</multiplier>
+			</plugin>
+		</gazebo>
+		<gazebo>
+			<plugin name="mimic_plugin" filename="libgazebo_mimic_plugin.so">
+				<joint>vergence_joint</joint>
+				<mimicJoint>l_eye_vergence_joint</mimicJoint>
+				<multiplier>-1.0</multiplier>
+			</plugin>
+		</gazebo>
+		<gazebo>
+			<plugin name="mimic_plugin" filename="libgazebo_mimic_plugin.so">
+				<joint>vergence_joint</joint>
+				<mimicJoint>r_eye_vergence_joint</mimicJoint>
+				<multiplier>1.0</multiplier>
+			</plugin>
+		</gazebo>
   </xacro:macro>
 </robot>

File: vizzy_description/urdf/head/head.transmission.xacro (robot description, xacro)
@@ -32,19 +32,55 @@
       </actuator>
     </transmission>
-    <transmission name="r_eye_pan_transmission">
+    <transmission name="version_transmission">
       <type>transmission_interface/SimpleTransmission</type>
-      <joint name="r_eye_pan_joint">
+      <joint name="version_joint">
         <hardwareInterface>EffortJointInterface</hardwareInterface>
       </joint>
-      <actuator name="r_eye_pan_motor">
+      <actuator name="version_motor">
+        <mechanicalReduction>100</mechanicalReduction>
+      </actuator>
+    </transmission>
+    <transmission name="l_eye_version_transmission">
+      <type>transmission_interface/SimpleTransmission</type>
+      <joint name="l_eye_version_joint">
+        <hardwareInterface>EffortJointInterface</hardwareInterface>
+      </joint>
+      <actuator name="l_eye_version_motor">
         <mechanicalReduction>1</mechanicalReduction>
       </actuator>
     </transmission>
-    <transmission name="l_eye_pan_transmission">
+    <transmission name="r_eye_version_transmission">
       <type>transmission_interface/SimpleTransmission</type>
-      <joint name="l_eye_pan_joint">
+      <joint name="r_eye_version_joint">
         <hardwareInterface>EffortJointInterface</hardwareInterface>
       </joint>
-      <actuator name="l_eye_pan_motor">
+      <actuator name="r_eye_version_motor">
+        <mechanicalReduction>1</mechanicalReduction>
+      </actuator>
+    </transmission>
+    <transmission name="vergence_transmission">
+      <type>transmission_interface/SimpleTransmission</type>
+      <joint name="vergence_joint">
+        <hardwareInterface>EffortJointInterface</hardwareInterface>
+      </joint>
+      <actuator name="vergence_motor">
+        <mechanicalReduction>100</mechanicalReduction>
+      </actuator>
+    </transmission>
+    <transmission name="l_eye_vergence_transmission">
+      <type>transmission_interface/SimpleTransmission</type>
+      <joint name="l_eye_vergence_joint">
+        <hardwareInterface>EffortJointInterface</hardwareInterface>
+      </joint>
+      <actuator name="l_eye_vergence_motor">
+        <mechanicalReduction>1</mechanicalReduction>
+      </actuator>
+    </transmission>
+    <transmission name="r_eye_vergence_transmission">
+      <type>transmission_interface/SimpleTransmission</type>
+      <joint name="r_eye_vergence_joint">
+        <hardwareInterface>EffortJointInterface</hardwareInterface>
+      </joint>
+      <actuator name="r_eye_vergence_motor">
         <mechanicalReduction>1</mechanicalReduction>
       </actuator>

File: vizzy_description/urdf/head/head.urdf.xacro (robot description, xacro)
@@ -60,6 +60,6 @@
     <axis
       xyz="0 0 1" />
-    <limit lower="-0.925024504" upper="0.925024504" effort="10" velocity="3" />
-    <dynamics damping="0.1"/>
+    <limit lower="-0.925024504" upper="0.925024504" effort="10.0" velocity="3" />
+    <dynamics damping="0.1" friction="0.1" />
   </joint>
   <link
@@ -115,6 +115,6 @@
     <axis
       xyz="0 0 1" />
-    <limit lower="-0.314159265" upper="0.645771823" effort="10" velocity="3" />
-    <dynamics damping="1.0"/>
+    <limit lower="-0.314159265" upper="0.645771823" effort="100.0" velocity="1.0" />
+    <dynamics damping="0.0" friction="0.0" />
   </joint>
   <link
@@ -170,9 +170,102 @@
     <axis
       xyz="0 0 1" />
-    <limit lower="-0.663225116" upper="0.663225116" effort="10" velocity="3" />
-    <dynamics damping="0.01"/>
-  </joint>
-  <link
-    name="r_eye_pan_link">
+    <limit lower="-0.663225116" upper="0.663225116" effort="10.0" velocity="3" />
+    <dynamics damping="0.1" friction="0.1" />
+  </joint>
+  <!-- version virtual link and joint -->
+  <link name="version_link">
+		<inertial>
+			<origin xyz="0 0 0"
+      rpy="0.0 0.0 0" />
+			<mass value="0.1"/>
+			<inertia
+				ixx="0.001" ixy="0.0" ixz="0.0"
+				iyy="0.001" iyz="0.0" izz="0.001"/>
+		</inertial>
+  </link>
+  <joint name="version_joint" type="revolute">
+    <origin xyz="0 0 0"       rpy="${M_PI/2.0} 0.0 0.369599135716446" />
+    <parent link="eyes_tilt_link" />
+    <child link="version_link" />
+    <axis  xyz="0 0 1" />
+    <limit lower="-0.698131" upper="0.698131" effort="10.0" velocity="0.2" />
+    <dynamics damping="1.0" friction="0.7" />
+  </joint>
+  <link name="l_eye_version_link">
+ 		<inertial>
+			<origin xyz="0 0 0" rpy="0 0 0"/>
+			<mass value="0.01"/>
+			<inertia
+				ixx="0.001" ixy="0.0" ixz="0.0"
+				iyy="0.001" iyz="0.0" izz="0.001"/>
+		</inertial>
+  </link>
+  <joint
+    name="l_eye_version_joint"
+    type="revolute">
+    <origin
+      xyz="0.0 0.0 0.102"
+      rpy="${M_PI/2.0} 0.0 0.369599135716446" />
+    <parent
+      link="eyes_tilt_link" />
+    <child
+      link="l_eye_version_link" />
+    <axis
+      xyz="0 0 1" />
+    <limit
+			lower="-1.0"
+			upper="1.0"
+      effort="1000.0"
+      velocity="0.2" />
+    <dynamics damping="0.1" friction="0.1" />
+    <mimic joint="version_joint" multiplier="1" offset="0"/>
+  </joint>
+  <link name="r_eye_version_link">
+ 		<inertial>
+			<origin xyz="0 0 0" rpy="0 0 0"/>
+			<mass value="0.01"/>
+			<inertia
+				ixx="0.001" ixy="0.0" ixz="0.0"
+				iyy="0.001" iyz="0.0" izz="0.001"/>
+		</inertial>
+  </link>
+  <joint
+    name="r_eye_version_joint"
+    type="revolute">
+    <origin
+      xyz="0.0 0.0 -0.102"
+      rpy="${M_PI/2.0} 0.0 0.369599135716446" />
+    <parent
+      link="eyes_tilt_link" />
+    <child
+      link="r_eye_version_link" />
+    <axis
+      xyz="0 0 1" />
+    <limit
+			lower="-1.0"
+			upper="1.0"
+      effort="1000.0"
+      velocity="0.2"/>
+    <dynamics damping="0.1" friction="0.1" />
+    <mimic joint="version_joint" multiplier="1" offset="0"/>
+  </joint>
+  <link name="vergence_link">
+ 		<inertial>
+			<origin xyz="0 0 0" rpy="0 0 0"/>
+			<mass value="0.1"/>
+			<inertia
+				ixx="0.001" ixy="0.0" ixz="0.0"
+				iyy="0.001" iyz="0.0" izz="0.001"/>
+		</inertial>
+  </link>
+  <joint name="vergence_joint" type="revolute">
+    <origin xyz="0.0 0.0 0.0" rpy="${M_PI/2.0} 0.0 0.369599135716446" />
+    <parent link="eyes_tilt_link" />
+    <child link="vergence_link" />
+    <axis  xyz="0 0 1" />
+    <limit lower="-0.698131" upper="0.698131" effort="10.0" velocity="0.2" />
+    <dynamics damping="1.0" friction="0.7" />
+  </joint>
+  <link name="r_eye_vergence_link">
     <inertial>
       <origin
@@ -214,17 +307,22 @@
   </link>
   <joint
-    name="r_eye_pan_joint"
-    type="revolute">
-    <origin
-      xyz="0.0 0.0 -0.102"
-      rpy="${M_PI/2.0} 0.0 0.369599135716446" />
-    <parent
-      link="eyes_tilt_link" />
-    <child
-      link="r_eye_pan_link" />
-    <axis
-      xyz="0 0 1" />
-    <limit lower="-0.698131" upper="0.698131" effort="10" velocity="3" />
-    <dynamics damping="0.1"/>
+    name="r_eye_vergence_joint"
+    type="revolute">
+    <origin
+      xyz="0.0 0.0 0.0"
+      rpy="0.0 0.0 0.0" />
+    <parent
+      link="r_eye_version_link" />
+    <child
+      link="r_eye_vergence_link" />
+    <axis
+      xyz="0 0 1" />
+		<limit
+			lower="-1.0"
+			upper="1.0"
+      effort="1000.0"
+      velocity="0.2"/>
+    <dynamics damping="0.1" friction="0.1" />
+    <mimic joint="vergence_joint" multiplier="1" offset="0"/>
   </joint>
   <link name="r_camera_link">
@@ -238,10 +336,9 @@
   <joint name="r_camera_joint" type="fixed">
     <origin xyz="0.0575 0.0 0.0" rpy="0.0 0.0 0.0" />
-    <parent link="r_eye_pan_link"/>
+    <parent link="r_eye_vergence_link"/>
     <child link="r_camera_link" />
   </joint>
-  <link
-    name="l_eye_pan_link">
-    <inertial>
+  <link name="l_eye_vergence_link">
+   <inertial>
       <origin
         xyz="0 0 -0.0200000000000069"
@@ -282,17 +379,22 @@
   </link>
   <joint
-    name="l_eye_pan_joint"
-    type="revolute">
-    <origin
-      xyz="0.0 0.0 0.102"
-      rpy="${M_PI/2.0} 0.0 0.369599135716446" />
-    <parent
-      link="eyes_tilt_link" />
-    <child
-      link="l_eye_pan_link" />
-    <axis
-      xyz="0 0 1" />
-    <limit lower="-0.698131" upper="0.698131" effort="10" velocity="3" />
-    <dynamics damping="0.1"/>
+    name="l_eye_vergence_joint"
+    type="revolute">
+    <origin
+      xyz="0 0 0"
+      rpy="0 0 0" />
+    <parent
+      link="l_eye_version_link" />
+    <child
+      link="l_eye_vergence_link" />
+    <axis
+      xyz="0 0 1" />
+    <limit
+			lower="-1.0"
+			upper="1.0"
+      effort="1000.0"
+      velocity="0.2" />
+    <dynamics damping="0.1" friction="0.1" />
+    <mimic joint="vergence_joint" multiplier="-1" offset="0"/>
   </joint>
   <link name="l_camera_link">
@@ -306,5 +408,5 @@
   <joint name="l_camera_joint" type="fixed">
     <origin xyz="0.0575 0.0 0.0" rpy="0.0 0.0 0.0" />
-    <parent link="l_eye_pan_link"/>
+    <parent link="l_eye_vergence_link"/>
     <child link="l_camera_link" />
   </joint>

File: vizzy_description/urdf/torso/torso.transmission.xacro (robot description, xacro)
@@ -11,5 +11,5 @@
       </joint>
       <actuator name="waist_motor">
-        <mechanicalReduction>1</mechanicalReduction>
+        <mechanicalReduction>100</mechanicalReduction>
       </actuator>
     </transmission>

File: vizzy_description/urdf/torso/torso.urdf.xacro (robot description, xacro)
@@ -61,6 +61,6 @@
     <axis
       xyz="0 0 1" />
-    <limit lower="-0.34906585" upper="0.34906585" effort="10" velocity="3" />
-    <dynamics damping="0.1"/>
+    <limit lower="-0.34906585" upper="0.34906585" effort="1000" velocity="10.0" />
+    <dynamics damping="1.0" friction="1.0"/>
   </joint>
   <!-- gazebo extensions -->

Commit message: added arms again

File: vizzy_description/robots/vizzy.urdf.xacro (robot description, xacro)
@@ -28,11 +28,11 @@
   <xacro:head name="head"/>
   <!-- instantiate left arm -->
-  <!--<xacro:left_arm name="left_arm" parent="waist_link" sufix="l" reflect="1">
+  <xacro:left_arm name="left_arm" parent="waist_link" sufix="l" reflect="1">
     <origin xyz="-0.01707 0.0 0.38145" rpy="0.0 0.0 0.0" />
-  </xacro:left_arm>-->
+  </xacro:left_arm>
   <!-- instantiate right arm -->
-  <!--<xacro:right_arm name="right_arm" parent="waist_link" sufix="r" reflect="1">
+  <xacro:right_arm name="right_arm" parent="waist_link" sufix="r" reflect="1">
     <origin xyz="-0.01707 0.0 0.38145" rpy="0.0 0.0 0.0" />
-  </xacro:right_arm>-->
+  </xacro:right_arm>
   <!-- instantiate hokuyo -->
   <xacro:hokuyo_mount name="nav_hokuyo" parent="base" length="${SENSOR_BEAM_LENGTH*INCH_TO_M}" ros_topic="scan" update_rate="10" min_angle="${-(5 * M_PI)/12}" max_angle="${(5 * M_PI)/12}">

File: vizzy_description/urdf/head/head.urdf.xacro (robot description, xacro)
@@ -264,5 +264,5 @@
     <child link="vergence_link" />
     <axis  xyz="0 0 1" />
-    <limit lower="-0.698131" upper="0.698131" effort="10.0" velocity="0.2" />
+    <limit lower="0.0" upper="0.698131" effort="10.0" velocity="0.2" />
     <dynamics damping="1.0" friction="0.7" />
   </joint>

Commit message: replaced Asus xtion with Intel realsense D435

File: vizzy_description/robots/vizzy.urdf.xacro (robot description, xacro)
@@ -17,6 +17,6 @@
   <!-- Hokuyo URG-04LX laser scanner -->
   <xacro:include filename="$(find vizzy_description)/urdf/sensors/hokuyo_04lx_laser.urdf.xacro"/>
-  <!-- TODO: Update Asus Xiton Live Pro -->
-  <xacro:include filename="$(find vizzy_description)/urdf/sensors/asus_camera.urdf.xacro"/>
+  <!-- RealSense D435 -->
+  <xacro:include filename="$(find vizzy_description)/urdf/sensors/_d435.urdf.xacro"/>
   <!-- Robot body -->
   <!-- Base -->
@@ -84,8 +84,7 @@
   <!-- Instantiate depth camera -->
   <xacro:unless value="$(arg disable_3d_sensor)">
-    <xacro:sensor_asus_xtion_pro name="asus_camera" parent="waist_link"
-      ros_topic="asus_camera">
-      <origin xyz="-0.08 0.16 0.02" rpy="${-M_PI/2} ${M_PI} ${-7*(M_PI/180)}"/>
-    </xacro:sensor_asus_xtion_pro>
+    <xacro:sensor_d435 name="realsense" parent="waist_link">
+      <origin xyz="-0.09516 0.143 0.0" rpy="${-M_PI/2} ${M_PI} 0"/> <!-- In the drawing z=0.158!!!-->
+    </xacro:sensor_d435>
   </xacro:unless>
   <!-- Instantiate plugins common to ROS and Yarp -->
