Commit message: finish reorganizing file structure

File: vizzy_description/urdf/arm/left_arm.gazebo.xacro (robot description, xacro)
@@ -1,12 +1,3 @@
 <?xml version="1.0"?>
 <robot xmlns:xacro="http://ros.org/wiki/xacro">
-  <xacro:macro name="left_arm_gazebo" params="name">
-    <!-- yarp plugin -->
-    <gazebo>
-      <plugin name="controlboard_left_arm" filename="libgazebo_yarp_controlboard.so">
-        <yarpConfigurationFile>model://media/conf/gazebo_vizzy_left_arm.ini</yarpConfigurationFile>
-        <initialConfiguration>0 0 0 0 0 0 0 0</initialConfiguration>
-      </plugin>
-    </gazebo>
-  </xacro:macro>
 </robot>

File: vizzy_description/urdf/arm/right_arm.gazebo.xacro (robot description, xacro)
@@ -1,12 +1,3 @@
 <?xml version="1.0"?>
 <robot xmlns:xacro="http://ros.org/wiki/xacro">
-  <xacro:macro name="right_arm_gazebo" params="name">
-  	<!-- yarp plugin -->
-    <gazebo>
-      <plugin name="controlboard_right_arm" filename="libgazebo_yarp_controlboard.so">
-        <yarpConfigurationFile>model://media/conf/gazebo_vizzy_right_arm.ini</yarpConfigurationFile>
-        <initialConfiguration>0 0 0 0 0 0 0 0</initialConfiguration>
-      </plugin>
-    </gazebo>
-  </xacro:macro>
 </robot>

File: vizzy_description/urdf/head/head.gazebo.xacro (robot description, xacro)
@@ -1,12 +1,5 @@
 <?xml version="1.0"?>
 <robot xmlns:xacro="http://ros.org/wiki/xacro">
-  <xacro:macro name="head_gazebo" params="name">
-    <!-- yarp plugin -->
-    <gazebo>
-      <plugin name="controlboard_head" filename="libgazebo_yarp_controlboard.so">
-        <yarpConfigurationFile>model://media/conf/gazebo_vizzy_head.ini</yarpConfigurationFile>
-        <initialConfiguration>0 0 0</initialConfiguration>
-      </plugin>
-    </gazebo>
+  <xacro:macro name="head_gazebo">
     <gazebo reference="neck_pan_link">
       <mu1>0.2</mu1>

File: vizzy_description/urdf/head/head.urdf.xacro (robot description, xacro)
@@ -310,5 +310,5 @@
   </joint>
     <!-- gazebo extensions -->
-    <xacro:head_gazebo name="${name}" />
+    <xacro:head_gazebo/>
     <xacro:head_transmissions />
   </xacro:macro>

File: vizzy_description/urdf/torso/torso.gazebo.xacro (robot description, xacro)
@@ -1,12 +1,5 @@
 <?xml version="1.0"?>
 <robot xmlns:xacro="http://ros.org/wiki/xacro">
-  <xacro:macro name="torso_gazebo" params="name">
-    <!-- yarp plugin -->
-    <gazebo>
-      <plugin name="controlboard_torso" filename="libgazebo_yarp_controlboard.so">
-        <yarpConfigurationFile>model://media/conf/gazebo_vizzy_torso.ini</yarpConfigurationFile>
-        <initialConfiguration>0</initialConfiguration>
-      </plugin>
-    </gazebo>
+  <xacro:macro name="torso_gazebo">
     <gazebo reference="waist_link">
       <gravity>false</gravity>

File: vizzy_description/urdf/torso/torso.urdf.xacro (robot description, xacro)
@@ -65,5 +65,5 @@
   </joint>
   <!-- gazebo extensions -->
-  <xacro:torso_gazebo name="${name}" />
+  <xacro:torso_gazebo/>
   <xacro:torso_transmissions/>
  </xacro:macro>
