Commit message: increased friction and damping factors of the joints

File: vizzy_description/urdf/arm/left_arm.urdf.xacro (robot description, xacro)
@@ -61,5 +61,5 @@
 		    xyz="0 0 1" />
 		  <limit lower="-0.314159265" upper="0.314159265" effort="10" velocity="3" />
-      <dynamics damping="0.1"/>
+    	<dynamics damping="1.0" friction="1000000.0" />
 		</joint>
 		<link
@@ -116,5 +116,5 @@
 		    xyz="0 0 1" />
 		  <limit lower="-1.30899694" upper="2.35619449" effort="10" velocity="3" />
-			<dynamics damping="0.1"/>
+    	<dynamics damping="1.0" friction="1000000.0" />
 		</joint>
 		<link
@@ -171,4 +171,5 @@
 		    xyz="0 0 1" />
 		  <limit lower="0" upper="1.30899694" effort="10" velocity="3" />
+    	<dynamics damping="1.0" friction="1000000.0" />
 		</joint>
 		<link
@@ -225,4 +226,5 @@
 		    xyz="0 0 1" />
 		  <limit lower="-1.48352986" upper="1.48352986" effort="10" velocity="3" />
+    	<dynamics damping="0.5" friction="1000000.0" />
 		</joint>
 		<link
@@ -279,4 +281,5 @@
 		    xyz="0 0 1" />
 		  <limit lower="0" upper="1.91986218" effort="10" velocity="3" />
+    	<dynamics damping="0.5" friction="1000000.0" />
 		</joint>
 		<link
@@ -333,4 +336,5 @@
 		    xyz="0 0 1" />
 		  <limit lower="-1.48352986" upper="1.48352986" effort="10" velocity="3" />
+    	<dynamics damping="0.1" friction="1000000.0" />
 		</joint>
 		<link
@@ -387,4 +391,5 @@
 		    xyz="0 0 1" />
 		  <limit lower="-0.610865238" upper="0.610865238" effort="10" velocity="3" />
+    	<dynamics damping="0.1" friction="1000000.0" />
 		</joint>
 		<link
@@ -441,4 +446,5 @@
 		    xyz="0 0 1" />
 		  <limit lower="-0.610865238" upper="0.610865238" effort="10" velocity="3" />
+    	<dynamics damping="0.1" friction="1000000.0" />
 		</joint>
 		<link name="l_palm_link">
@@ -454,4 +460,5 @@
 		  <parent link="l_wrist_flection_link"/>
 		  <child link="l_palm_link" />
+    	<dynamics damping="0.1" friction="1000000.0" />
 		</joint>
 		<!-- gazebo extensions -->

File: vizzy_description/urdf/arm/right_arm.urdf.xacro (robot description, xacro)
@@ -61,4 +61,5 @@
 		    xyz="0 0 1" />
 		  <limit lower="-0.314159265" upper="0.314159265" effort="10" velocity="3" />
+    	<dynamics damping="1.0" friction="1000000.0" />
 		</joint>
 		<link
@@ -115,4 +116,5 @@
 		    xyz="0 0 1" />
 		  <limit lower="-1.30899694" upper="2.35619449" effort="10" velocity="3" />
+    	<dynamics damping="1.0" friction="1000000.0" />
 		</joint>
 		<link
@@ -169,4 +171,5 @@
 		    xyz="0 0 1" />
 		  <limit lower="0" upper="1.30899694" effort="10" velocity="3" />
+    	<dynamics damping="1.0" friction="1000000.0" />
 		</joint>
 		<link
@@ -223,4 +226,5 @@
 		    xyz="0 0 1" />
 		  <limit lower="-1.48352986" upper="1.48352986" effort="10" velocity="3" />
+    	<dynamics damping="0.5" friction="1000000.0" />
 		</joint>
 		<link
@@ -277,4 +281,5 @@
 		    xyz="0 0 1" />
 		  <limit lower="0" upper="1.91986218" effort="10" velocity="3" />
+    	<dynamics damping="0.5" friction="1000000.0" />
 		</joint>
 		<link
@@ -331,4 +336,5 @@
 		    xyz="0 0 1" />
 		  <limit lower="-1.48352986" upper="1.48352986" effort="10" velocity="3" />
+    	<dynamics damping="0.1" friction="1000000.0" />
 		</joint>
 		<link
@@ -385,4 +391,5 @@
 		    xyz="0 0 1" />
 		  <limit lower="-0.610865238" upper="0.610865238" effort="10" velocity="3" />
+    	<dynamics damping="0.1" friction="1000000.0" />
 		</joint>
 		<link
@@ -439,4 +446,5 @@
 		    xyz="0 0 1" />
 		  <limit lower="-0.610865238" upper="0.610865238" effort="10" velocity="3" />
+    	<dynamics damping="0.1" friction="1000000.0" />
 		</joint>
 		<link name="r_palm_link">
@@ -452,4 +460,5 @@
 		  <parent link="r_wrist_flection_link"/>
 		  <child link="r_palm_link" />
+    	<dynamics damping="0.1" friction="1000000.0" />
 		</joint>
     <!-- gazebo extensions -->

File: vizzy_description/urdf/head/head.ros.urdf.xacro (robot description, xacro)
@@ -116,5 +116,5 @@
       xyz="0 0 1" />
     <limit lower="-0.314159265" upper="0.645771823" effort="100.0" velocity="1.0" />
-    <dynamics damping="0.0" friction="0.0" />
+    <dynamics damping="10.0" friction="1000000.0" />
   </joint>
   <link
@@ -171,5 +171,5 @@
       xyz="0 0 1" />
     <limit lower="-0.663225116" upper="0.663225116" effort="10.0" velocity="3" />
-    <dynamics damping="0.1" friction="0.1" />
+    <dynamics damping="0.1" friction="10.0" />
   </joint>
   <!-- eyes center virtual link and joint -->

File: vizzy_description/urdf/head/head.urdf.xacro (robot description, xacro)
@@ -61,5 +61,5 @@
       xyz="0 0 1" />
     <limit lower="-0.925024504" upper="0.925024504" effort="10.0" velocity="3" />
-    <dynamics damping="0.1" friction="0.1" />
+    <dynamics damping="10.0" friction="100.0" />
   </joint>
   <link
@@ -116,5 +116,5 @@
       xyz="0 0 1" />
     <limit lower="-0.314159265" upper="0.645771823" effort="100.0" velocity="1.0" />
-    <dynamics damping="0.0" friction="0.0" />
+    <dynamics damping="10.0" friction="100.0" />
   </joint>
   <link
@@ -171,5 +171,5 @@
       xyz="0 0 1" />
     <limit lower="-0.663225116" upper="0.663225116" effort="10.0" velocity="3" />
-    <dynamics damping="0.1" friction="0.1" />
+    <dynamics damping="10.0" friction="100.0" />
   </joint>
   <!-- version virtual link and joint -->

File: vizzy_description/urdf/torso/torso.urdf.xacro (robot description, xacro)
@@ -62,5 +62,5 @@
       xyz="0 0 1" />
     <limit lower="-0.34906585" upper="0.34906585" effort="${3863H024C_motor_max_effort}" velocity="${3863H024C_motor_max_velocitiy*DEG_TO_RAD}" />
-    <dynamics damping="1.0" friction="1.0"/>
+    <dynamics damping="20.0" friction="1000000.0"/>
   </joint>
   <!-- gazebo extensions -->

Commit message: Removed damping from both arms

File: vizzy_description/urdf/arm/left_arm.urdf.xacro (robot description, xacro)
@@ -61,5 +61,4 @@
 		    xyz="0 0 1" />
 		  <limit lower="-0.314159265" upper="0.314159265" effort="10" velocity="3" />
-    	<dynamics damping="1.0" friction="1000000.0" />
 		</joint>
 		<link
@@ -116,5 +115,4 @@
 		    xyz="0 0 1" />
 		  <limit lower="-1.30899694" upper="2.35619449" effort="10" velocity="3" />
-    	<dynamics damping="1.0" friction="1000000.0" />
 		</joint>
 		<link
@@ -171,5 +169,4 @@
 		    xyz="0 0 1" />
 		  <limit lower="0" upper="1.30899694" effort="10" velocity="3" />
-    	<dynamics damping="1.0" friction="1000000.0" />
 		</joint>
 		<link
@@ -226,5 +223,4 @@
 		    xyz="0 0 1" />
 		  <limit lower="-1.48352986" upper="1.48352986" effort="10" velocity="3" />
-    	<dynamics damping="0.5" friction="1000000.0" />
 		</joint>
 		<link
@@ -281,5 +277,4 @@
 		    xyz="0 0 1" />
 		  <limit lower="0" upper="1.91986218" effort="10" velocity="3" />
-    	<dynamics damping="0.5" friction="1000000.0" />
 		</joint>
 		<link
@@ -336,5 +331,4 @@
 		    xyz="0 0 1" />
 		  <limit lower="-1.48352986" upper="1.48352986" effort="10" velocity="3" />
-    	<dynamics damping="0.1" friction="1000000.0" />
 		</joint>
 		<link
@@ -391,5 +385,4 @@
 		    xyz="0 0 1" />
 		  <limit lower="-0.610865238" upper="0.610865238" effort="10" velocity="3" />
-    	<dynamics damping="0.1" friction="1000000.0" />
 		</joint>
 		<link
@@ -446,5 +439,4 @@
 		    xyz="0 0 1" />
 		  <limit lower="-0.610865238" upper="0.610865238" effort="10" velocity="3" />
-    	<dynamics damping="0.1" friction="1000000.0" />
 		</joint>
 		<link name="l_palm_link">
@@ -460,5 +452,4 @@
 		  <parent link="l_wrist_flection_link"/>
 		  <child link="l_palm_link" />
-    	<dynamics damping="0.1" friction="1000000.0" />
 		</joint>
 		<!-- gazebo extensions -->

File: vizzy_description/urdf/arm/right_arm.urdf.xacro (robot description, xacro)
@@ -61,5 +61,4 @@
 		    xyz="0 0 1" />
 		  <limit lower="-0.314159265" upper="0.314159265" effort="10" velocity="3" />
-    	<dynamics damping="1.0" friction="1000000.0" />
 		</joint>
 		<link
@@ -116,5 +115,4 @@
 		    xyz="0 0 1" />
 		  <limit lower="-1.30899694" upper="2.35619449" effort="10" velocity="3" />
-    	<dynamics damping="1.0" friction="1000000.0" />
 		</joint>
 		<link
@@ -171,5 +169,4 @@
 		    xyz="0 0 1" />
 		  <limit lower="0" upper="1.30899694" effort="10" velocity="3" />
-    	<dynamics damping="1.0" friction="1000000.0" />
 		</joint>
 		<link
@@ -226,5 +223,4 @@
 		    xyz="0 0 1" />
 		  <limit lower="-1.48352986" upper="1.48352986" effort="10" velocity="3" />
-    	<dynamics damping="0.5" friction="1000000.0" />
 		</joint>
 		<link
@@ -281,5 +277,4 @@
 		    xyz="0 0 1" />
 		  <limit lower="0" upper="1.91986218" effort="10" velocity="3" />
-    	<dynamics damping="0.5" friction="1000000.0" />
 		</joint>
 		<link
@@ -336,5 +331,4 @@
 		    xyz="0 0 1" />
 		  <limit lower="-1.48352986" upper="1.48352986" effort="10" velocity="3" />
-    	<dynamics damping="0.1" friction="1000000.0" />
 		</joint>
 		<link
@@ -391,5 +385,4 @@
 		    xyz="0 0 1" />
 		  <limit lower="-0.610865238" upper="0.610865238" effort="10" velocity="3" />
-    	<dynamics damping="0.1" friction="1000000.0" />
 		</joint>
 		<link
@@ -446,5 +439,4 @@
 		    xyz="0 0 1" />
 		  <limit lower="-0.610865238" upper="0.610865238" effort="10" velocity="3" />
-    	<dynamics damping="0.1" friction="1000000.0" />
 		</joint>
 		<link name="r_palm_link">
@@ -460,5 +452,4 @@
 		  <parent link="r_wrist_flection_link"/>
 		  <child link="r_palm_link" />
-    	<dynamics damping="0.1" friction="1000000.0" />
 		</joint>
     <!-- gazebo extensions -->
