Commit message: [vizzy_description] comment with Temporary fix for index finger encoder record

File: vizzy_description/urdf/arm/arm.urdf.xacro (robot description, xacro)
@@ -334,5 +334,6 @@
           reflect="${reflect}" rpy="${wrist_flection_l_rpy}" prefix="${prefix}"/>
       </link>
-      <joint name="${prefix}_wrist_flection_joint"
+	<!-- <joint name="${prefix}_index_flection" Temporary fix for index finger encoder record-->
+       <joint name="${prefix}_wrist_flection_joint"
         type="revolute">
         <origin
