Commit message: minor changes

File: vizzy_description/urdf/torso/torso.transmission.xacro (robot description, xacro)
@@ -11,5 +11,5 @@
       </joint>
       <actuator name="waist_motor">
-        <mechanicalReduction>100</mechanicalReduction>
+        <mechanicalReduction>${3863H024C_motor_transmission_reduction}</mechanicalReduction>
       </actuator>
     </transmission>

File: vizzy_description/urdf/torso/torso.urdf.xacro (robot description, xacro)
@@ -61,5 +61,5 @@
     <axis
       xyz="0 0 1" />
-    <limit lower="-0.34906585" upper="0.34906585" effort="1000" velocity="10.0" />
+    <limit lower="-0.34906585" upper="0.34906585" effort="${3863H024C_motor_max_effort}" velocity="${3863H024C_motor_max_velocitiy*DEG_TO_RAD}" />
     <dynamics damping="1.0" friction="1.0"/>
   </joint>
