Commit message: fixes....

File: vizzy_description/urdf/head/head.ros.gazebo.xacro (robot description, xacro)
@@ -50,24 +50,10 @@
     </gazebo>
  		<gazebo reference="neck_pan_joint">
-			<kd value="1.0" />
-			<kp value="1000000.0" />
-			<fudgeFactor value="1.0" />
-			<provideFeedback value="true"/>
 		</gazebo>
  		<gazebo reference="neck_tilt_joint">
-			<kd value="1.0" />
-			<kp value="1000000.0" />
-			<fudgeFactor value="1.0" />
-			<provideFeedback value="true"/>
 		</gazebo>
  		<gazebo reference="eyes_tilt_joint">
-			<kd value="1.0" />
-			<kp value="1000000.0" />
-			<fudgeFactor value="1.0" />
-			<provideFeedback value="true"/>
 		</gazebo>
  		<gazebo reference="version_joint">
-  		<stopKd value="1000000.0" />
-  		<stopKp value="1000000.0" />
 		</gazebo>
  		<!--<gazebo reference="l_eye_version_joint">

File: vizzy_description/urdf/head/head.ros.urdf.xacro (robot description, xacro)
@@ -61,5 +61,4 @@
       xyz="0 0 1" />
     <limit lower="-0.925024504" upper="0.925024504" effort="10.0" velocity="5.0" />
-    <dynamics damping="0.1" friction="0.1" />
   </joint>
   <link
@@ -116,5 +115,4 @@
       xyz="0 0 1" />
     <limit lower="-0.314159265" upper="0.645771823" effort="100.0" velocity="5.0" />
-    <dynamics damping="10.0" friction="1000000.0" />
   </joint>
   <link
@@ -171,5 +169,4 @@
       xyz="0 0 1" />
     <limit lower="-0.663225116" upper="0.663225116" effort="10.0" velocity="5.0" />
-    <dynamics damping="0.1" friction="10.0" />
   </joint>
   <!-- eyes center virtual link and joint -->

File: vizzy_description/urdf/torso/torso.gazebo.xacro (robot description, xacro)
@@ -12,5 +12,5 @@
 			<fudgeFactor value="1.0" />
 			<provideFeedback value="true"/>
-  		<dampingFactor>0.7</dampingFactor>
+  		        <dampingFactor>0.7</dampingFactor>
 		</gazebo>
   </xacro:macro>
