Commit message: fixes

File: vizzy_description/urdf/head/head.urdf.xacro (robot description, xacro)
@@ -61,5 +61,4 @@
       xyz="0 0 1" />
     <limit lower="-0.925024504" upper="0.925024504" effort="10.0" velocity="3" />
-    <dynamics damping="10.0" friction="100.0" />
   </joint>
   <link
@@ -116,5 +115,4 @@
       xyz="0 0 1" />
     <limit lower="-0.314159265" upper="0.645771823" effort="100.0" velocity="1.0" />
-    <dynamics damping="10.0" friction="100.0" />
   </joint>
   <link
@@ -171,5 +169,4 @@
       xyz="0 0 1" />
     <limit lower="-0.663225116" upper="0.663225116" effort="10.0" velocity="3" />
-    <dynamics damping="10.0" friction="100.0" />
   </joint>
   <!-- version virtual link and joint -->
@@ -190,5 +187,4 @@
     <axis  xyz="0 0 1" />
     <limit lower="-0.698131" upper="0.698131" effort="10.0" velocity="0.2" />
-    <dynamics damping="1.0" friction="0.7" />
   </joint>
   <link name="l_eye_version_link">
@@ -218,5 +214,4 @@
       effort="1000.0"
       velocity="0.2" />
-    <dynamics damping="0.1" friction="0.1" />
     <mimic joint="version_joint" multiplier="1" offset="0"/>
   </joint>
@@ -247,5 +242,4 @@
       effort="1000.0"
       velocity="0.2"/>
-    <dynamics damping="0.1" friction="0.1" />
     <mimic joint="version_joint" multiplier="1" offset="0"/>
   </joint>
@@ -265,5 +259,4 @@
     <axis  xyz="0 0 1" />
     <limit lower="0.0" upper="0.698131" effort="10.0" velocity="0.2" />
-    <dynamics damping="1.0" friction="0.7" />
   </joint>
   <link name="r_eye_vergence_link">
@@ -323,5 +316,4 @@
       effort="1000.0"
       velocity="0.2"/>
-    <dynamics damping="0.1" friction="0.1" />
     <mimic joint="vergence_joint" multiplier="1" offset="0"/>
   </joint>
@@ -408,5 +400,4 @@
       effort="1000.0"
       velocity="0.2" />
-    <dynamics damping="0.1" friction="0.1" />
     <mimic joint="vergence_joint" multiplier="-1" offset="0"/>
   </joint>

File: vizzy_description/urdf/head/head.yarp.urdf.xacro (robot description, xacro)
@@ -61,5 +61,4 @@
       xyz="0 0 1" />
     <limit lower="-0.925024504" upper="0.925024504" effort="10" velocity="3" />
-    <dynamics damping="0.1"/>
   </joint>
   <link
@@ -116,5 +115,4 @@
       xyz="0 0 1" />
     <limit lower="-0.314159265" upper="0.645771823" effort="10" velocity="3" />
-    <dynamics damping="1.0"/>
   </joint>
   <link
@@ -171,5 +169,4 @@
       xyz="0 0 1" />
     <limit lower="-0.663225116" upper="0.663225116" effort="10" velocity="3" />
-    <dynamics damping="0.01"/>
   </joint>
   <link
@@ -226,5 +223,4 @@
       xyz="0 0 1" />
     <limit lower="-0.698131" upper="0.698131" effort="10" velocity="3" />
-    <dynamics damping="0.1"/>
   </joint>
   <link name="r_camera_link">
@@ -294,5 +290,4 @@
       xyz="0 0 1" />
     <limit lower="-0.698131" upper="0.698131" effort="10" velocity="3" />
-    <dynamics damping="0.1"/>
   </joint>
   <link name="l_camera_link">

File: vizzy_description/urdf/torso/torso.gazebo.xacro (robot description, xacro)
@@ -12,5 +12,4 @@
 			<fudgeFactor value="1.0" />
 			<provideFeedback value="true"/>
-  		        <dampingFactor>0.7</dampingFactor>
 		</gazebo>
   </xacro:macro>

File: vizzy_description/urdf/torso/torso.urdf.xacro (robot description, xacro)
@@ -62,5 +62,4 @@
       xyz="0 0 1" />
     <limit lower="-0.34906585" upper="0.34906585" effort="${3863H024C_motor_max_effort}" velocity="${3863H024C_motor_max_velocitiy*DEG_TO_RAD}" />
-    <dynamics damping="20.0" friction="1000000.0"/>
   </joint>
   <!-- gazebo extensions -->
