Commit message: increased physics engine number of iterations in gazebo

File: vizzy_description/urdf/head/head.gazebo.xacro (robot description, xacro)
@@ -3,20 +3,8 @@
   <xacro:macro name="head_gazebo">
     <gazebo reference="neck_pan_link">
-      <mu1>0.2</mu1>
-      <mu2>0.2</mu2>
- 			<kp value="100.0" />
-			<kd value="1.0" />
     </gazebo>
     <gazebo reference="neck_tilt_link">
-      <mu1>0.2</mu1>
-      <mu2>0.2</mu2>
- 			<kp value="100.0" />
-			<kd value="1.0" />
     </gazebo>
     <gazebo reference="eyes_tilt_link">
-      <mu1>0.2</mu1>
-      <mu2>0.2</mu2>
- 			<kp value="100.0" />
-			<kd value="1.0" />
     </gazebo>
     <gazebo reference="version_link">
@@ -27,64 +15,19 @@
     </gazebo>
     <gazebo reference="vergence_link">
-      <gravity value="false"/>
-      <mu1>0.2</mu1>
-      <mu2>0.2</mu2>
- 			<kp value="100.0" />
-			<kd value="1.0" />
     </gazebo>
 		 <gazebo reference="r_eye_vergence_link">
-      <mu1>0.2</mu1>
-      <mu2>0.2</mu2>
- 			<kp value="100.0" />
-			<kd value="1.0" />
     </gazebo>
     <gazebo reference="l_eye_vergence_link">
-      <mu1>0.2</mu1>
-      <mu2>0.2</mu2>
- 			<kp value="100.0" />
-			<kd value="1.0" />
     </gazebo>
  		<gazebo reference="neck_pan_joint">
-			<kd value="1.0" />
-			<kp value="100.0" />
-			<fudgeFactor value="1.0" />
-			<provideFeedback value="true"/>
 		</gazebo>
  		<gazebo reference="neck_tilt_joint">
-			<kd value="1.0" />
-			<kp value="100.0" />
-			<fudgeFactor value="1.0" />
-			<provideFeedback value="true"/>
 		</gazebo>
  		<gazebo reference="eyes_tilt_joint">
-			<kd value="1.0" />
-			<kp value="100.0" />
-			<fudgeFactor value="1.0" />
-			<provideFeedback value="true"/>
 		</gazebo>
  		<gazebo reference="version_joint">
-  		<stopKd value="100.0" />
-  		<stopKp value="100.0" />
 		</gazebo>
- 		<!--<gazebo reference="l_eye_version_joint">
-  		<stopKd value="100.0" />
-  		<stopKp value="100.0" />
+ 		<gazebo reference="vergence_joint">
 		</gazebo>
- 		<gazebo reference="r_eye_version_joint">
-  		<stopKd value="100.0" />
-  		<stopKp value="100.0" />
-		</gazebo>-->
- 		<gazebo reference="vergence_joint">
-  		<stopKd value="100.0" />
-  		<stopKp value="100.0" />
-		</gazebo>
- 		<!--<gazebo reference="l_eye_vergence_joint">
-  		<stopKd value="100.0" />
-  		<stopKp value="100.0" />
-		</gazebo>
- 		<gazebo reference="r_eye_vergence_joint">
-  		<stopKd value="100.0" />
-  		<stopKp value="100.0" />
-		</gazebo>-->
 		<gazebo>
 			<plugin name="mimic_plugin" filename="libgazebo_mimic_plugin.so">

File: vizzy_description/urdf/head/head.ros.urdf.xacro (robot description, xacro)
@@ -278,5 +278,5 @@
  		<inertial>
 			<origin xyz="0 0 0" rpy="0 0 0"/>
-			<mass value="0.001"/>
+			<mass value="0.01"/>
 			<inertia
 				ixx="0.001" ixy="0.0" ixz="0.0"
