Commit message: removed damping factors from the eyes, which were messing with the controllers

File: vizzy_description/urdf/head/head.ros.urdf.xacro (robot description, xacro)
@@ -221,5 +221,4 @@
     <axis  xyz="0 0 1" />
     <limit lower="-0.698131" upper="0.698131" effort="10.0" velocity="5.0" />
-    <dynamics damping="1.0" friction="0.7" />
   </joint>
   <link name="l_eye_version_link">
@@ -249,5 +248,4 @@
       effort="1000.0"
       velocity="5.0" />
-    <dynamics damping="0.1" friction="0.1" />
     <mimic joint="version_joint" multiplier="1" offset="0"/>
   </joint>
@@ -278,5 +276,4 @@
       effort="1000.0"
       velocity="5.0"/>
-    <dynamics damping="0.1" friction="0.1" />
     <mimic joint="version_joint" multiplier="1" offset="0"/>
   </joint>
@@ -296,5 +293,4 @@
     <axis  xyz="0 0 1" />
     <limit lower="0.0" upper="0.698131" effort="10.0" velocity="5.0" />
-    <dynamics damping="1.0" friction="0.7" />
   </joint>
   <link name="r_eye_vergence_link">
@@ -354,5 +350,4 @@
       effort="1000.0"
       velocity="5.0"/>
-    <dynamics damping="0.1" friction="0.1" />
     <mimic joint="vergence_joint" multiplier="1" offset="0"/>
   </joint>
@@ -439,5 +434,4 @@
       effort="1000.0"
       velocity="5.0" />
-    <dynamics damping="0.1" friction="0.1" />
     <mimic joint="vergence_joint" multiplier="-1" offset="0"/>
   </joint>

Commit message: fix

File: vizzy_description/urdf/head/head.ros.urdf.xacro (robot description, xacro)
@@ -459,4 +459,21 @@
     <child link="l_camera_vision_link" />
   </joint>
+  <!-- eyes center virtual link and joint -->
+  <link name="ego_frame">
+    <inertial>
+      <origin xyz="0 0 0" rpy="0.0 0.0 0" />
+      <mass value="0.001"/>
+      <inertia
+        ixx="0.001" ixy="0.0" ixz="0.0"
+        iyy="0.001" iyz="0.0" izz="0.001"/>
+    </inertial>
+  </link>
+  <joint name="ego_joint" type="fixed">
+    <origin
+      xyz="0.0 0.370 0.0"
+      rpy="0.0 ${M_PI/2.0} ${M_PI}" />
+    <parent link="waist_link"/>
+    <child link="ego_frame" />
+  </joint>
     <!-- gazebo extensions -->
     <xacro:head_gazebo/>

Commit message: changed mimic scale of the vergence joint to the right value (0.5 instead of 1), but still the output is not correct

File: vizzy_description/urdf/head/head.ros.urdf.xacro (robot description, xacro)
@@ -348,5 +348,5 @@
       effort="1000.0"
       velocity="5.0"/>
-    <mimic joint="vergence_joint" multiplier="1" offset="0"/>
+    <mimic joint="vergence_joint" multiplier="0.5" offset="0"/>
   </joint>
   <link name="r_camera_link">
@@ -432,5 +432,5 @@
       effort="1000.0"
       velocity="5.0" />
-    <mimic joint="vergence_joint" multiplier="-1" offset="0"/>
+    <mimic joint="vergence_joint" multiplier="-0.5" offset="0"/>
   </joint>
   <link name="l_camera_link">

File: vizzy_description/urdf/head/head.urdf.xacro (robot description, xacro)
@@ -316,5 +316,5 @@
       effort="1000.0"
       velocity="0.2"/>
-    <mimic joint="vergence_joint" multiplier="1" offset="0"/>
+    <mimic joint="vergence_joint" multiplier="0.5" offset="0"/>
   </joint>
   <link name="r_camera_link">
@@ -400,5 +400,5 @@
       effort="1000.0"
       velocity="0.2" />
-    <mimic joint="vergence_joint" multiplier="-1" offset="0"/>
+    <mimic joint="vergence_joint" multiplier="-0.5" offset="0"/>
   </joint>
   <link name="l_camera_link">

Commit message: added extra frame for convenience

File: vizzy_description/urdf/head/head.ros.urdf.xacro (robot description, xacro)
@@ -477,4 +477,20 @@
     <child link="ego_frame" />
   </joint>
+  <link name="head_origin_frame">
+    <inertial>
+      <origin xyz="0 0 0" rpy="0.0 0.0 0" />
+      <mass value="0.001"/>
+      <inertia
+        ixx="0.001" ixy="0.0" ixz="0.0"
+        iyy="0.001" iyz="0.0" izz="0.001"/>
+    </inertial>
+  </link>
+  <joint name="head_origin_joint" type="fixed">
+    <origin
+      xyz="0.0 -0.04755 0.0"
+      rpy="0.0 -${M_PI/2.0} 0.0" />
+    <parent link="neck_tilt_link"/>
+    <child link="head_origin_frame" />
+  </joint>
     <!-- gazebo extensions -->
     <xacro:head_gazebo/>
