Commit message: working on attention results

File: vizzy_description/urdf/base/base.gazebo.xacro (robot description, xacro)
@@ -11,34 +11,34 @@
     </gazebo>
     <gazebo reference="b_wheel_base_link">
-      <mu1>0.2</mu1>
-      <mu2>0.2</mu2>
+      <mu1>10000</mu1>
+      <mu2>10000</mu2>
     </gazebo>
     <gazebo reference="b_wheel_link">
-      <mu1>0.2</mu1>
-      <mu2>0.2</mu2>
+      <mu1>10000</mu1>
+      <mu2>10000</mu2>
     </gazebo>
     <gazebo reference="f_wheel_base_link">
-      <mu1>0.2</mu1>
-      <mu2>0.2</mu2>
+      <mu1>10000</mu1>
+      <mu2>10000</mu2>
     </gazebo>
     <gazebo reference="f_wheel_link">
-      <mu1>0.2</mu1>
-      <mu2>0.2</mu2>
+      <mu1>10000</mu1>
+      <mu2>10000</mu2>
     </gazebo>
     <gazebo reference="l_wheel_base_link">
-      <mu1>0.2</mu1>
-      <mu2>0.2</mu2>
+      <mu1>10000</mu1>
+      <mu2>10000</mu2>
     </gazebo>
     <gazebo reference="l_wheel_link">
-      <mu1>0.2</mu1>
-      <mu2>0.2</mu2>
+      <mu1>10000</mu1>
+      <mu2>10000</mu2>
     </gazebo>
     <gazebo reference="r_wheel_base_link">
-      <mu1>0.2</mu1>
-      <mu2>0.2</mu2>
+      <mu1>10000</mu1>
+      <mu2>10000</mu2>
     </gazebo>
     <gazebo reference="r_wheel_link">
-      <mu1>0.2</mu1>
-      <mu2>0.2</mu2>
+      <mu1>10000</mu1>
+      <mu2>10000</mu2>
     </gazebo>
   </xacro:macro>

File: vizzy_description/urdf/head/head.ros.gazebo.xacro (robot description, xacro)
@@ -3,26 +3,10 @@
   <xacro:macro name="head_gazebo">
     <gazebo reference="neck_pan_link">
-      <mu1>0.2</mu1>
-      <mu2>0.2</mu2>
- 			<kp value="1000000.0" />
-			<kd value="1.0" />
     </gazebo>
     <gazebo reference="neck_tilt_link">
-      <mu1>0.2</mu1>
-      <mu2>0.2</mu2>
- 			<kp value="1000000.0" />
-			<kd value="1.0" />
     </gazebo>
     <gazebo reference="eyes_tilt_link">
-      <mu1>0.2</mu1>
-      <mu2>0.2</mu2>
- 			<kp value="1000000.0" />
-			<kd value="1.0" />
     </gazebo>
     <gazebo reference="version_link">
-      <mu1>0.2</mu1>
-      <mu2>0.2</mu2>
- 			<kp value="1.0" />
-			<kd value="1.0" />
     </gazebo>
     <gazebo reference="r_eye_version_link">
@@ -31,21 +15,8 @@
     </gazebo>
     <gazebo reference="vergence_link">
-      <gravity value="false"/>
-      <mu1>0.2</mu1>
-      <mu2>0.2</mu2>
- 			<kp value="1.0" />
-			<kd value="1.0" />
     </gazebo>
-		 <gazebo reference="r_eye_vergence_link">
-      <mu1>0.2</mu1>
-      <mu2>0.2</mu2>
- 			<kp value="1000000.0" />
-			<kd value="1.0" />
+  <gazebo reference="r_eye_vergence_link">
     </gazebo>
     <gazebo reference="l_eye_vergence_link">
-      <mu1>0.2</mu1>
-      <mu2>0.2</mu2>
- 			<kp value="1000000.0" />
-			<kd value="1.0" />
     </gazebo>
  		<gazebo reference="neck_pan_joint">
@@ -57,24 +28,6 @@
  		<gazebo reference="version_joint">
 		</gazebo>
- 		<!--<gazebo reference="l_eye_version_joint">
-  		<stopKd value="1000000.0" />
-  		<stopKp value="1000000.0" />
+ 		<gazebo reference="vergence_joint">
 		</gazebo>
- 		<gazebo reference="r_eye_version_joint">
-  		<stopKd value="1000000.0" />
-  		<stopKp value="1000000.0" />
-		</gazebo>-->
- 		<gazebo reference="vergence_joint">
-  		<stopKd value="1000000.0" />
-  		<stopKp value="1000000.0" />
-		</gazebo>
- 		<!--<gazebo reference="l_eye_vergence_joint">
-  		<stopKd value="1000000.0" />
-  		<stopKp value="1000000.0" />
-		</gazebo>
- 		<gazebo reference="r_eye_vergence_joint">
-  		<stopKd value="1000000.0" />
-  		<stopKp value="1000000.0" />
-		</gazebo>-->
 		<gazebo>
 			<plugin name="mimic_plugin" filename="libgazebo_mimic_plugin.so">

File: vizzy_description/urdf/head/head.ros.urdf.xacro (robot description, xacro)
@@ -405,7 +405,7 @@
     </visual>
     <collision>
-      <origin
-        xyz="0 0 -0.0200000000000069"
-        rpy="0 0 1.5708" />
+ 	<origin
+        xyz="0.010 0.0 0.003"
+        rpy="0.0 ${M_PI} ${-M_PI/2}" />
       <geometry>
         <mesh
