Commit message: minor changes

File: vizzy_description/urdf/simple_base/base.urdf.xacro (robot description, xacro)
@@ -16,12 +16,12 @@
   <link name="base_link">
    <inertial>
-     <origin xyz="0 0 0.25" rpy="0 0 0"/>
+     <origin xyz="0 0 0.125" rpy="0 0 0"/>
      <mass value="1"/>
      <inertia ixx="100"  ixy="0"  ixz="0" iyy="100" iyz="0" izz="100" />
    </inertial>
    <visual>
-     <origin xyz="0 0 0.25" rpy="0 0 0" />
+     <origin xyz="0 0 0.125" rpy="0 0 0" />
      <geometry>
-       <cylinder radius="0.05" length="0.25"/>
+       <cylinder radius="0.01" length="0.25"/>
      </geometry>
      <material name="Cyan">
@@ -30,7 +30,7 @@
    </visual>
    <collision>
-     <origin xyz="0 0 0.25" rpy="0 0 0"/>
+     <origin xyz="0 0 0.125" rpy="0 0 0"/>
      <geometry>
-       <cylinder radius="0.05" length="0.25"/>
+       <cylinder radius="0.01" length="0.25"/>
      </geometry>
    </collision>
