Commit message: finished right hand urdf

File: vizzy_description/urdf/hand/right_hand.urdf.xacro (robot description, xacro)
@@ -174,15 +174,15 @@
     <inertial>
       <origin
-        xyz="-0.0065949 -2.2728E-05 0.013411"
-        rpy="0 0 0" />
-      <mass
-        value="0.0093855" />
-      <inertia
-        ixx="5.7614E-07"
-        ixy="5.3191E-10"
-        ixz="-3.8097E-11"
-        iyy="5.3414E-07"
-        iyz="3.9566E-09"
-        izz="3.158E-07" />
+        xyz="-0.00659486836575895 -2.27276594980388E-05 0.0134108525654478"
+        rpy="0 0 0" />
+      <mass
+        value="0.00938546678393586" />
+      <inertia
+        ixx="5.76143838934573E-07"
+        ixy="5.31905829930291E-10"
+        ixz="-3.8097259604833E-11"
+        iyy="5.34143788531799E-07"
+        iyz="3.95661158120478E-09"
+        izz="3.15804741452118E-07" />
     </inertial>
     <visual>
@@ -197,5 +197,5 @@
         name="">
         <color
-          rgba="0.89804 0.91765 0.92941 1" />
+          rgba="0.898039215686275 0.917647058823529 0.929411764705882 1" />
       </material>
     </visual>
@@ -696,5 +696,5 @@
     <inertial>
       <origin
-        xyz="-1.3326E-05 3.9324E-05 0.0033395"
+        xyz="-1.3326E-05 3.9324E-05 0.01634"
         rpy="0 0 0" />
       <mass
@@ -736,6 +736,6 @@
     type="revolute">
     <origin
-      xyz="0 0.0028 0.046"
-      rpy="-1.7831E-12 -6.1062E-16 -4.7716E-13" />
+      xyz="0 0.0031104 0.032985"
+      rpy="-0.0094057 -6.9111E-15 -2.4286E-17" />
     <parent
       link="thumb_phal_2_link" />
