Commit message: overall repository cleaning

File: vizzy_description/plugins/ros.gazebo.xacro (robot description, xacro)
@@ -1,6 +1,6 @@
 <?xml version="1.0"?>
 <root xmlns:xacro="http://ros.org/wiki/xacro">
-  <!-- head, torso and arms controllers plugin -->
-  <xacro:macro name="ros_control_gazebo">
+	<!-- head, torso and arms controllers plugin -->
+	<xacro:macro name="ros_control_gazebo">
     <gazebo>
 	    <plugin name="gazebo_ros_control" filename="libgazebo_ros_control.so">
@@ -13,5 +13,5 @@
 	  <gazebo>
       <plugin name="differential_drive_controller" filename="libgazebo_ros_diff_drive.so">
-        <leftJoint>l_wheel_joint</leftJoint>
+      	<leftJoint>l_wheel_joint</leftJoint>
         <rightJoint>r_wheel_joint</rightJoint>
         <wheelSeparation>0.4580</wheelSeparation>
@@ -26,4 +26,5 @@
     </gazebo>
   </xacro:macro>
+  <!-- camera plugin -->
   <xacro:macro name="camera_plugin" params="name prefix">
     <gazebo reference="${prefix}_camera_link">

File: vizzy_description/robots/vizzy.urdf.xacro (robot description, xacro)
@@ -1,7 +1,5 @@
 <?xml version="1.0"?>
 <robot  name="vizzy" xmlns:xacro="http://ros.org/wiki/xacro" >
-  <!-- - - - - - - - - - - - - - - - - - - - - - - - - - - - - - - - - - - - - - - -->
-  <!--  The following include files set up definitions of parts of the robot body  -->
-  <!-- - - - - - - - - - - - - - - - - - - - - - - - - - - - - - - - - - - - - - - -->
+  <!-- The following include files set up definitions of parts of the robot body  -->
   <!-- misc common stuff -->
   <xacro:include filename="$(find vizzy_description)/urdf/common.urdf.xacro" />
@@ -18,7 +16,5 @@
   <!-- right arm -->
   <xacro:include filename="$(find vizzy_description)/urdf/arm/right_arm.urdf.xacro" />
-  <!-- - - - - - - - - - - - - - - - - - - - - - - - - -  -->
 	<!-- The following include files contain gazebo plugins -->
-  <!-- - - - - - - - - - - - - - - - - - - - - - - - - -  -->
   <!-- ROS -->
   <xacro:include filename="$(find vizzy_description)/plugins/ros.gazebo.xacro" />
@@ -41,6 +37,5 @@
   <!-- instantiate hokuyo -->
   <xacro:hokuyo_mount name="nav_hokuyo" parent="base" length="${SENSOR_BEAM_LENGTH*INCH_TO_M}" ros_topic="scan" update_rate="10" min_angle="${-(5 * M_PI)/12}" max_angle="${(5 * M_PI)/12}">
-    <origin xyz="-0.05 0.14
- 0.15" rpy="${-M_PI/2} ${-M_PI/2} 3.14" />
+    <origin xyz="-0.05 0.14 0.15" rpy="${-M_PI/2} ${-M_PI/2} 3.14" />
   </xacro:hokuyo_mount>
   <!-- instantiate common ROS and Yarp plugins -->

Commit message: minor identation changes

File: vizzy_description/plugins/ros.gazebo.xacro (robot description, xacro)
@@ -1,17 +1,17 @@
 <?xml version="1.0"?>
 <root xmlns:xacro="http://ros.org/wiki/xacro">
-	<!-- head, torso and arms controllers plugin -->
-	<xacro:macro name="ros_control_gazebo">
+  <!-- head, torso and arms controllers plugin -->
+  <xacro:macro name="ros_control_gazebo">
     <gazebo>
-	    <plugin name="gazebo_ros_control" filename="libgazebo_ros_control.so">
-		    <robotNamespace>/vizzy</robotNamespace>
-		  </plugin>
+      <plugin name="gazebo_ros_control" filename="libgazebo_ros_control.so">
+        <robotNamespace>/vizzy</robotNamespace>
+      </plugin>
     </gazebo>
   </xacro:macro>
   <!-- base controller plugin -->
   <xacro:macro name="ros_differential_drive_gazebo">
-	  <gazebo>
+    <gazebo>
       <plugin name="differential_drive_controller" filename="libgazebo_ros_diff_drive.so">
-      	<leftJoint>l_wheel_joint</leftJoint>
+        <leftJoint>l_wheel_joint</leftJoint>
         <rightJoint>r_wheel_joint</rightJoint>
         <wheelSeparation>0.4580</wheelSeparation>
@@ -29,43 +29,43 @@
   <xacro:macro name="camera_plugin" params="name prefix">
     <gazebo reference="${prefix}_camera_link">
-		  <sensor type="camera" name="${prefix}_camera">
-				<update_rate>30.0</update_rate>
-				<camera name="head">
-				  <horizontal_fov>1.4912</horizontal_fov>
-				  <image>
-				    <width>320</width>
-				    <height>240</height>
-				    <format>R8G8B8</format>
-				  </image>
-				  <clip>
-				    <near>0.02</near>
-				    <far>300</far>
-				  </clip>
-				  <noise>
-				    <type>gaussian</type>
-				    <!-- Noise is sampled independently per pixel on each frame.
-				         That pixel's noise value is added to each of its color
-				         channels, which at that point lie in the range [0,1]. -->
-				    <mean>0.0</mean>
-				    <stddev>0.007</stddev>
-				  </noise>
-				</camera>
-				<plugin name="camera_controller" filename="libgazebo_ros_camera.so">
-				  <alwaysOn>true</alwaysOn>
-				  <updateRate>30.0</updateRate>
-				  <cameraName>vizzy/${prefix}_camera</cameraName>
-				  <imageTopicName>image_raw</imageTopicName>
-				  <cameraInfoTopicName>camera_info</cameraInfoTopicName>
-				  <frameName>${prefix}_camera_link</frameName>
-				  <distortion>
-				    <k1>-0.4738</k1>
-				    <k2>0.190309</k2>
-				    <k3>0.0</k3>
-				    <p1>-0.000375676</p1>
-				    <p2>-0.000663688</p2>
-				    <center> 0.4809  0.4887</center>
-				  </distortion>
-				</plugin>
-			</sensor>
+      <sensor type="camera" name="${prefix}_camera">
+        <update_rate>30.0</update_rate>
+        <camera name="head">
+          <horizontal_fov>1.4912</horizontal_fov>
+          <image>
+            <width>320</width>
+            <height>240</height>
+            <format>R8G8B8</format>
+          </image>
+          <clip>
+            <near>0.02</near>
+            <far>300</far>
+          </clip>
+          <noise>
+            <type>gaussian</type>
+            <!-- Noise is sampled independently per pixel on each frame.
+                That pixel's noise value is added to each of its color
+                channels, which at that point lie in the range [0,1]. -->
+            <mean>0.0</mean>
+            <stddev>0.007</stddev>
+          </noise>
+        </camera>
+        <plugin name="camera_controller" filename="libgazebo_ros_camera.so">
+          <alwaysOn>true</alwaysOn>
+          <updateRate>30.0</updateRate>
+          <cameraName>vizzy/${prefix}_camera</cameraName>
+          <imageTopicName>image_raw</imageTopicName>
+          <cameraInfoTopicName>camera_info</cameraInfoTopicName>
+          <frameName>${prefix}_camera_link</frameName>
+          <distortion>
+            <k1>-0.4738</k1>
+            <k2>0.190309</k2>
+            <k3>0.0</k3>
+            <p1>-0.000375676</p1>
+            <p2>-0.000663688</p2>
+            <center> 0.4809  0.4887</center>
+          </distortion>
+        </plugin>
+      </sensor>
     </gazebo>
   </xacro:macro>

Commit message: fixed problem with TFs

File: vizzy_description/plugins/ros.gazebo.xacro (robot description, xacro)
@@ -18,5 +18,5 @@
         <wheelDiameter>0.2410</wheelDiameter>
         <torque>20</torque>
-        <commandTopic>cmd_vel</commandTopic>
+        <commandTopic>vizzy/cmd_vel</commandTopic>
         <odometryTopic>odom</odometryTopic>
         <odometryFrame>odom</odometryFrame>

File: vizzy_description/robots/vizzy.urdf.xacro (robot description, xacro)
@@ -28,9 +28,9 @@
   <xacro:head name="head"/>
   <!-- instantiate left arm -->
-  <xacro:left_arm name="left_arm" parent="M0" sufix="l" reflect="1">
+  <xacro:left_arm name="left_arm" parent="waist_link" sufix="l" reflect="1">
     <origin xyz="-0.01707 0.0 0.38145" rpy="0.0 0.0 0.0" />
   </xacro:left_arm>
   <!-- instantiate right arm -->
-  <xacro:right_arm name="right_arm" parent="M0" sufix="r" reflect="1">
+  <xacro:right_arm name="right_arm" parent="waist_link" sufix="r" reflect="1">
     <origin xyz="-0.01707 0.0 0.38145" rpy="0.0 0.0 0.0" />
   </xacro:right_arm>

File: vizzy_description/urdf/arm/left_arm.transmission.xacro (robot description, xacro)
@@ -20,4 +20,13 @@
       </joint>
       <actuator name="l_shoulder_flection_motor">
+        <mechanicalReduction>1</mechanicalReduction>
+      </actuator>
+    </transmission>
+    <transmission name="l_shoulder_abduction_transmission">
+      <type>transmission_interface/SimpleTransmission</type>
+      <joint name="l_shoulder_abduction_joint">
+        <hardwareInterface>EffortJointInterface</hardwareInterface>
+      </joint>
+      <actuator name="l_shoulder_abduction_motor">
         <mechanicalReduction>1</mechanicalReduction>
       </actuator>

File: vizzy_description/urdf/arm/left_arm.urdf.xacro (robot description, xacro)
@@ -61,4 +61,5 @@
 		    xyz="0 0 1" />
 		  <limit lower="-0.314159265" upper="0.314159265" effort="10" velocity="3" />
+      <dynamics damping="0.1"/>
 		</joint>
 		<link
@@ -115,4 +116,5 @@
 		    xyz="0 0 1" />
 		  <limit lower="-1.30899694" upper="2.35619449" effort="10" velocity="3" />
+			<dynamics damping="0.1"/>
 		</joint>
 		<link

File: vizzy_description/urdf/base/base.gazebo.xacro (robot description, xacro)
@@ -1,33 +1,45 @@
 <?xml version="1.0"?>
 <robot xmlns:xacro="http://ros.org/wiki/xacro">
-  <xacro:macro name="base_gazebo" params="name">
-    <!--<gazebo reference="b_wheel_link">
-      <turnGravityOff>false</turnGravityOff>
+  <xacro:macro name="base_gazebo">
+    <gazebo reference="base_link">
+      <mu1>0.2</mu1>
+      <mu2>0.2</mu2>
     </gazebo>
-    <gazebo reference="b_wheel_joint">
-      <stopKd value="1.0" />
-      <stopKp value="1000.0" />
+    <gazebo reference="base_footprint">
+      <mu1>0.2</mu1>
+      <mu2>0.2</mu2>
     </gazebo>
     <gazebo reference="b_wheel_base_link">
-      <turnGravityOff>false</turnGravityOff>
+      <mu1>0.2</mu1>
+      <mu2>0.2</mu2>
     </gazebo>
-    <gazebo reference="b_wheel_base_joint">
-      <stopKd value="1.0" />
-      <stopKp value="1000.0" />
+    <gazebo reference="b_wheel_link">
+      <mu1>0.2</mu1>
+      <mu2>0.2</mu2>
+    </gazebo>
+    <gazebo reference="f_wheel_base_link">
+      <mu1>0.2</mu1>
+      <mu2>0.2</mu2>
     </gazebo>
     <gazebo reference="f_wheel_link">
-      <turnGravityOff>false</turnGravityOff>
+      <mu1>0.2</mu1>
+      <mu2>0.2</mu2>
     </gazebo>
-    <gazebo reference="f_wheel_joint">
-      <stopKd value="1.0" />
-      <stopKp value="1000.0" />
+    <gazebo reference="l_wheel_base_link">
+      <mu1>0.2</mu1>
+      <mu2>0.2</mu2>
     </gazebo>
-    <gazebo reference="f_wheel_base_link">
-      <turnGravityOff>false</turnGravityOff>
+    <gazebo reference="l_wheel_link">
+      <mu1>0.2</mu1>
+      <mu2>0.2</mu2>
     </gazebo>
-    <gazebo reference="f_wheel_base_joint">
-      <stopKd value="1.0" />
-      <stopKp value="1000.0" />
-    </gazebo>-->
+    <gazebo reference="r_wheel_base_link">
+      <mu1>0.2</mu1>
+      <mu2>0.2</mu2>
+    </gazebo>
+    <gazebo reference="r_wheel_link">
+      <mu1>0.2</mu1>
+      <mu2>0.2</mu2>
+    </gazebo>
   </xacro:macro>
 </robot>

File: vizzy_description/urdf/base/base.transmission.xacro (robot description, xacro)
@@ -4,74 +4,56 @@
        xmlns:interface="http://playerstage.sourceforge.net/gazebo/xmlschema/#interface"
        xmlns:xacro="http://ros.org/wiki/xacro">
-  <xacro:macro name="right_arm_transmissions">
-    <transmission name="r_shoulder_scapula_transmission">
+  <xacro:macro name="base_transmissions">
+    <transmission name="f_wheel_transmission">
       <type>transmission_interface/SimpleTransmission</type>
-      <joint name="r_shoulder_scapula_joint">
+      <joint name="f_wheel_joint">
         <hardwareInterface>EffortJointInterface</hardwareInterface>
       </joint>
-      <actuator name="r_shoulder_scapula_motor">
+      <actuator name="f_wheel_motor">
         <mechanicalReduction>1</mechanicalReduction>
       </actuator>
     </transmission>
-    <transmission name="r_shoulder_flection_transmission">
+    <transmission name="f_wheel_base_transmission">
       <type>transmission_interface/SimpleTransmission</type>
-      <joint name="r_shoulder_flection_joint">
+      <joint name="f_wheel_base_joint">
         <hardwareInterface>EffortJointInterface</hardwareInterface>
       </joint>
-      <actuator name="r_shoulder_flection_motor">
+      <actuator name="f_wheel_base_motor">
         <mechanicalReduction>1</mechanicalReduction>
       </actuator>
     </transmission>
-    <transmission name="r_shoulder_abduction_transmission">
+    <transmission name="b_wheel_transmission">
       <type>transmission_interface/SimpleTransmission</type>
-      <joint name="r_shoulder_abduction_joint">
+      <joint name="b_wheel_joint">
         <hardwareInterface>EffortJointInterface</hardwareInterface>
       </joint>
-      <actuator name="r_shoulder_abduction_motor">
+      <actuator name="b_wheel_motor">
         <mechanicalReduction>1</mechanicalReduction>
       </actuator>
     </transmission>
-    <transmission name="r_shoulder_rotation_transmission">
+    <transmission name="b_wheel_base_transmission">
       <type>transmission_interface/SimpleTransmission</type>
-      <joint name="r_shoulder_rotation_joint">
+      <joint name="b_wheel_base_joint">
         <hardwareInterface>EffortJointInterface</hardwareInterface>
       </joint>
-      <actuator name="r_shoulder_rotation_motor">
+      <actuator name="b_wheel_base_motor">
         <mechanicalReduction>1</mechanicalReduction>
       </actuator>
     </transmission>
-    <transmission name="r_elbow_flection_transmission">
+    <transmission name="r_wheel_transmission">
       <type>transmission_interface/SimpleTransmission</type>
-      <joint name="r_elbow_flection_joint">
+      <joint name="r_wheel_joint">
         <hardwareInterface>EffortJointInterface</hardwareInterface>
       </joint>
-      <actuator name="r_elbow_flection_motor">
+      <actuator name="r_wheel_base_motor">
         <mechanicalReduction>1</mechanicalReduction>
       </actuator>
     </transmission>
-    <transmission name="r_forearm_pronation_transmission">
+    <transmission name="l_wheel_transmission">
       <type>transmission_interface/SimpleTransmission</type>
-      <joint name="r_forearm_pronation_joint">
+      <joint name="l_wheel_joint">
         <hardwareInterface>EffortJointInterface</hardwareInterface>
       </joint>
-      <actuator name="r_forearm_pronation_motor">
-        <mechanicalReduction>1</mechanicalReduction>
-      </actuator>
-    </transmission>
-    <transmission name="r_wrist_abduction_transmission">
-      <type>transmission_interface/SimpleTransmission</type>
-      <joint name="r_wrist_abduction_joint">
-        <hardwareInterface>EffortJointInterface</hardwareInterface>
-      </joint>
-      <actuator name="r_wrist_abduction_motor">
-        <mechanicalReduction>1</mechanicalReduction>
-      </actuator>
-    </transmission>
-    <transmission name="r_wrist_flection_transmission">
-      <type>transmission_interface/SimpleTransmission</type>
-      <joint name="r_wrist_flection_joint">
-        <hardwareInterface>EffortJointInterface</hardwareInterface>
-      </joint>
-      <actuator name="r_wrist_flection_motor">
+      <actuator name="l_wheel_base_motor">
         <mechanicalReduction>1</mechanicalReduction>
       </actuator>

File: vizzy_description/urdf/base/base.urdf.xacro (robot description, xacro)
@@ -7,5 +7,5 @@
        sensor and controller plugin specifications -->
  <xacro:include filename="$(find vizzy_description)/urdf/base/base.gazebo.xacro" />
- <!--<xacro:include filename="$(find vizzy_description)/urdf/base/base.transmission.xacro" />-->
+ <xacro:include filename="$(find vizzy_description)/urdf/base/base.transmission.xacro" />
  <xacro:macro name="base" params="name">
   <!-- root link, on the ground just below the robot origin -->
@@ -115,5 +115,4 @@
     <axis
       xyz="0 0 1" />
-    <dynamics damping="0.1"/>
   </joint>
   <link
@@ -222,5 +221,4 @@
     <axis
       xyz="0 0 1" />
-    <dynamics damping="0.1"/>
   </joint>
   <link
@@ -384,6 +382,6 @@
   </joint>
   <!-- gazebo extensions -->
-  <xacro:base_gazebo name="${name}" />
-  <!--<xacro:base_transmissions/>-->
+  <xacro:base_gazebo/>
+  <xacro:base_transmissions/>
  </xacro:macro>
 </robot>

Commit message: launch with move_base option working

File: vizzy_description/plugins/ros.gazebo.xacro (robot description, xacro)
@@ -13,6 +13,7 @@
     <gazebo>
       <plugin name="differential_drive_controller" filename="libgazebo_ros_diff_drive.so">
-        <leftJoint>l_wheel_joint</leftJoint>
-        <rightJoint>r_wheel_joint</rightJoint>
+        <!-- hack -->
+        <leftJoint>r_wheel_joint</leftJoint>
+        <rightJoint>l_wheel_joint</rightJoint>
         <wheelSeparation>0.4580</wheelSeparation>
         <wheelDiameter>0.2410</wheelDiameter>

File: vizzy_description/urdf/base/base.urdf.xacro (robot description, xacro)
@@ -19,5 +19,5 @@
   </link>
   <joint name="base_footprint_joint" type="fixed">
-   <origin xyz="0 0 0" rpy="0 0 0" />
+   <origin xyz="0.0 0.0 0.0" rpy="0.0 0.0 ${M_PI}" />
    <parent link="base_footprint"/>
    <child link="base_link" />

Commit message: deleted unused files and added extra fixed virtual joint for convenience

File: vizzy_description/plugins/ros.gazebo.xacro (robot description, xacro)
@@ -49,5 +49,5 @@
                 channels, which at that point lie in the range [0,1]. -->
             <mean>0.0</mean>
-            <stddev>0.007</stddev>
+            <stddev>0.000</stddev>
           </noise>
         </camera>

File: vizzy_description/urdf/head/head.ros.urdf.xacro (robot description, xacro)
@@ -173,4 +173,20 @@
     <dynamics damping="0.1" friction="0.1" />
   </joint>
+  <!-- eyes center virtual link and joint -->
+  <link name="eyes_center_link">
+		<inertial>
+			<origin xyz="0 0 0"
+      rpy="0.0 0.0 0" />
+			<mass value="0.1"/>
+			<inertia
+				ixx="0.001" ixy="0.0" ixz="0.0"
+				iyy="0.001" iyz="0.0" izz="0.001"/>
+		</inertial>
+  </link>
+  <joint name="eyes_center_joint" type="fixed">
+    <origin xyz="0 0 0"       rpy="${M_PI/2.0} 0.0 0.369599135716446" />
+    <parent link="eyes_tilt_link" />
+    <child link="eyes_center_link" />
+  </joint>
   <!-- version virtual link and joint -->
   <link name="version_link">
@@ -185,6 +201,6 @@
   </link>
   <joint name="version_joint" type="revolute">
-    <origin xyz="0 0 0"       rpy="${M_PI/2.0} 0.0 0.369599135716446" />
-    <parent link="eyes_tilt_link" />
+    <origin xyz="0 0 0"       rpy="0 0 0" />
+    <parent link="eyes_center_link" />
     <child link="version_link" />
     <axis  xyz="0 0 1" />
@@ -205,8 +221,8 @@
     type="revolute">
     <origin
-      xyz="0.0 0.0 0.102"
-      rpy="${M_PI/2.0} 0.0 0.369599135716446" />
-    <parent
-      link="eyes_tilt_link" />
+      xyz="0.0 0.102 0.0"
+      rpy="0 0 0" />
+    <parent
+      link="eyes_center_link" />
     <child
       link="l_eye_version_link" />
@@ -234,8 +250,8 @@
     type="revolute">
     <origin
-      xyz="0.0 0.0 -0.102"
-      rpy="${M_PI/2.0} 0.0 0.369599135716446" />
-    <parent
-      link="eyes_tilt_link" />
+      xyz="0.0 -0.102 0.0"
+      rpy="0 0.0 0" />
+    <parent
+      link="eyes_center_link" />
     <child
       link="r_eye_version_link" />
@@ -260,6 +276,6 @@
   </link>
   <joint name="vergence_joint" type="revolute">
-    <origin xyz="0.0 0.0 0.0" rpy="${M_PI/2.0} 0.0 0.369599135716446" />
-    <parent link="eyes_tilt_link" />
+    <origin xyz="0.0 0.0 0.0" rpy="0 0.0 0" />
+    <parent link="eyes_center_link" />
     <child link="vergence_link" />
     <axis  xyz="0 0 1" />

Commit message: working on stereo

File: vizzy_description/plugins/ros.gazebo.xacro (robot description, xacro)
@@ -59,5 +59,5 @@
           <cameraInfoTopicName>camera_info</cameraInfoTopicName>
           <frameName>${prefix}_camera_link</frameName>
-          <distortion>
+          <!--<distortion>
             <k1>-0.4738</k1>
             <k2>0.190309</k2>
@@ -66,5 +66,5 @@
             <p2>-0.000663688</p2>
             <center> 0.4809  0.4887</center>
-          </distortion>
+          </distortion>-->
         </plugin>
       </sensor>

File: vizzy_description/urdf/head/head.ros.urdf.xacro (robot description, xacro)
@@ -184,4 +184,19 @@
 		</inertial>
   </link>
+  <joint name="eyes_center_vision_joint" type="fixed">
+    <origin xyz="0 0 0"       rpy="${-M_PI/2} 0.0 ${-M_PI/2}" />
+    <parent link="eyes_center_link" />
+    <child link="eyes_center_vision_link" />
+  </joint>
+  <link name="eyes_center_vision_link">
+		<inertial>
+			<origin xyz="0 0 0"
+      rpy="0.0 0.0 0" />
+			<mass value="0.1"/>
+			<inertia
+				ixx="0.001" ixy="0.0" ixz="0.0"
+				iyy="0.001" iyz="0.0" izz="0.001"/>
+		</inertial>
+  </link>
   <joint name="eyes_center_joint" type="fixed">
     <origin xyz="0 0 0"       rpy="${M_PI/2.0} 0.0 0.369599135716446" />
@@ -355,4 +370,17 @@
     <child link="r_camera_link" />
   </joint>
+  <link name="r_camera_vision_link">
+   <visual>
+      <origin xyz="0 0 0" rpy="0 0 0" />
+      <geometry>
+        <box size="0.001 0.001 0.001" />
+      </geometry>
+    </visual>
+  </link>
+  <joint name="r_camera_vision_joint" type="fixed">
+    <origin xyz="0.0 0.0 0.0" rpy="${-M_PI/2} 0.0 ${-M_PI/2}" />
+    <parent link="r_camera_link"/>
+    <child link="r_camera_vision_link" />
+  </joint>
   <link name="l_eye_vergence_link">
    <inertial>
@@ -427,4 +455,17 @@
     <child link="l_camera_link" />
   </joint>
+  <link name="l_camera_vision_link">
+   <visual>
+      <origin xyz="0 0 0" rpy="0 0 0" />
+      <geometry>
+        <box size="0.001 0.001 0.001" />
+      </geometry>
+    </visual>
+  </link>
+  <joint name="l_camera_vision_joint" type="fixed">
+    <origin xyz="0.0 0.0 0.0" rpy="${-M_PI/2} 0.0 ${-M_PI/2}" />
+    <parent link="l_camera_link"/>
+    <child link="l_camera_vision_link" />
+  </joint>
     <!-- gazebo extensions -->
     <xacro:head_gazebo/>

File: vizzy_description/urdf/head/head.urdf.xacro (robot description, xacro)
@@ -339,4 +339,17 @@
     <child link="r_camera_link" />
   </joint>
+  <link name="r_camera_vision_link">
+   <visual>
+      <origin xyz="0 0 0" rpy="0 0 0" />
+      <geometry>
+        <box size="0.001 0.001 0.001" />
+      </geometry>
+    </visual>
+  </link>
+  <joint name="r_camera_vision_joint" type="fixed">
+    <origin xyz="0.0 0.0 0.0" rpy="0.0 ${M_PI/2} 0.0" />
+    <parent link="r_camera_link"/>
+    <child link="r_camera_vision_link" />
+  </joint>
   <link name="l_eye_vergence_link">
    <inertial>
@@ -411,4 +424,17 @@
     <child link="l_camera_link" />
   </joint>
+  <link name="l_camera_vision_link">
+   <visual>
+      <origin xyz="0 0 0" rpy="0 0 0" />
+      <geometry>
+        <box size="0.001 0.001 0.001" />
+      </geometry>
+    </visual>
+  </link>
+  <joint name="l_camera_vision_joint" type="fixed">
+    <origin xyz="0.0 0.0 0.0" rpy="0.0 ${M_PI/2} 0.0" />
+    <parent link="l_camera_link"/>
+    <child link="l_camera_vision_link" />
+  </joint>
     <!-- gazebo extensions -->
     <xacro:head_gazebo/>
