Commit message: moveit

File: vizzy_description/plugins/ros.gazebo.xacro (robot description, xacro)
@@ -35,6 +35,8 @@
           <horizontal_fov>1.4912</horizontal_fov>
           <image>
-            <width>320</width>
-            <height>240</height>
+            <!--<width>320</width>
+            <height>240</height>-->
+            <width>300</width>
+            <height>300</height>
             <format>R8G8B8</format>
           </image>

File: vizzy_description/robots/vizzy.urdf.xacro (robot description, xacro)
@@ -1,4 +1,5 @@
 <?xml version="1.0"?>
 <robot  name="vizzy" xmlns:xacro="http://ros.org/wiki/xacro" >
+	<xacro:arg name="use_yarp" default="false"/>
   <!-- The following include files set up definitions of parts of the robot body  -->
   <!-- misc common stuff -->

File: vizzy_description/urdf/arm/left_arm.transmission.xacro (robot description, xacro)
@@ -8,5 +8,5 @@
       <type>transmission_interface/SimpleTransmission</type>
       <joint name="l_shoulder_scapula_joint">
-        <hardwareInterface>EffortJointInterface</hardwareInterface>
+        <hardwareInterface>VelocityJointInterface</hardwareInterface>
       </joint>
       <actuator name="l_shoulder_scapula_motor">
@@ -17,5 +17,5 @@
       <type>transmission_interface/SimpleTransmission</type>
       <joint name="l_shoulder_flection_joint">
-        <hardwareInterface>EffortJointInterface</hardwareInterface>
+        <hardwareInterface>VelocityJointInterface</hardwareInterface>
       </joint>
       <actuator name="l_shoulder_flection_motor">
@@ -26,5 +26,5 @@
       <type>transmission_interface/SimpleTransmission</type>
       <joint name="l_shoulder_abduction_joint">
-        <hardwareInterface>EffortJointInterface</hardwareInterface>
+        <hardwareInterface>VelocityJointInterface</hardwareInterface>
       </joint>
       <actuator name="l_shoulder_abduction_motor">
@@ -35,5 +35,5 @@
       <type>transmission_interface/SimpleTransmission</type>
       <joint name="l_shoulder_rotation_joint">
-        <hardwareInterface>EffortJointInterface</hardwareInterface>
+        <hardwareInterface>VelocityJointInterface</hardwareInterface>
       </joint>
       <actuator name="l_shoulder_rotation_motor">
@@ -44,5 +44,5 @@
       <type>transmission_interface/SimpleTransmission</type>
       <joint name="l_elbow_flection_joint">
-        <hardwareInterface>EffortJointInterface</hardwareInterface>
+        <hardwareInterface>VelocityJointInterface</hardwareInterface>
       </joint>
       <actuator name="l_elbow_flection_motor">
@@ -53,5 +53,5 @@
       <type>transmission_interface/SimpleTransmission</type>
       <joint name="l_forearm_pronation_joint">
-        <hardwareInterface>EffortJointInterface</hardwareInterface>
+        <hardwareInterface>VelocityJointInterface</hardwareInterface>
       </joint>
       <actuator name="l_forearm_pronation_motor">
@@ -62,5 +62,5 @@
       <type>transmission_interface/SimpleTransmission</type>
       <joint name="l_wrist_abduction_joint">
-        <hardwareInterface>EffortJointInterface</hardwareInterface>
+        <hardwareInterface>VelocityJointInterface</hardwareInterface>
       </joint>
       <actuator name="l_wrist_abduction_motor">
@@ -71,5 +71,5 @@
       <type>transmission_interface/SimpleTransmission</type>
       <joint name="l_wrist_flection_joint">
-        <hardwareInterface>EffortJointInterface</hardwareInterface>
+        <hardwareInterface>VelocityJointInterface</hardwareInterface>
       </joint>
       <actuator name="l_wrist_flection_motor">

File: vizzy_description/urdf/arm/right_arm.transmission.xacro (robot description, xacro)
@@ -8,5 +8,5 @@
       <type>transmission_interface/SimpleTransmission</type>
       <joint name="r_shoulder_scapula_joint">
-        <hardwareInterface>EffortJointInterface</hardwareInterface>
+        <hardwareInterface>VelocityJointInterface</hardwareInterface>
       </joint>
       <actuator name="r_shoulder_scapula_motor">
@@ -17,5 +17,5 @@
       <type>transmission_interface/SimpleTransmission</type>
       <joint name="r_shoulder_flection_joint">
-        <hardwareInterface>EffortJointInterface</hardwareInterface>
+        <hardwareInterface>VelocityJointInterface</hardwareInterface>
       </joint>
       <actuator name="r_shoulder_flection_motor">
@@ -26,5 +26,5 @@
       <type>transmission_interface/SimpleTransmission</type>
       <joint name="r_shoulder_abduction_joint">
-        <hardwareInterface>EffortJointInterface</hardwareInterface>
+        <hardwareInterface>VelocityJointInterface</hardwareInterface>
       </joint>
       <actuator name="r_shoulder_abduction_motor">
@@ -35,5 +35,5 @@
       <type>transmission_interface/SimpleTransmission</type>
       <joint name="r_shoulder_rotation_joint">
-        <hardwareInterface>EffortJointInterface</hardwareInterface>
+        <hardwareInterface>VelocityJointInterface</hardwareInterface>
       </joint>
       <actuator name="r_shoulder_rotation_motor">
@@ -44,5 +44,5 @@
       <type>transmission_interface/SimpleTransmission</type>
       <joint name="r_elbow_flection_joint">
-        <hardwareInterface>EffortJointInterface</hardwareInterface>
+        <hardwareInterface>VelocityJointInterface</hardwareInterface>
       </joint>
       <actuator name="r_elbow_flection_motor">
@@ -53,5 +53,5 @@
       <type>transmission_interface/SimpleTransmission</type>
       <joint name="r_forearm_pronation_joint">
-        <hardwareInterface>EffortJointInterface</hardwareInterface>
+        <hardwareInterface>VelocityJointInterface</hardwareInterface>
       </joint>
       <actuator name="r_forearm_pronation_motor">
@@ -62,5 +62,5 @@
       <type>transmission_interface/SimpleTransmission</type>
       <joint name="r_wrist_abduction_joint">
-        <hardwareInterface>EffortJointInterface</hardwareInterface>
+        <hardwareInterface>VelocityJointInterface</hardwareInterface>
       </joint>
       <actuator name="r_wrist_abduction_motor">
@@ -71,5 +71,5 @@
       <type>transmission_interface/SimpleTransmission</type>
       <joint name="r_wrist_flection_joint">
-        <hardwareInterface>EffortJointInterface</hardwareInterface>
+        <hardwareInterface>VelocityJointInterface</hardwareInterface>
       </joint>
       <actuator name="r_wrist_flection_motor">

File: vizzy_description/urdf/head/head.gazebo.xacro (robot description, xacro)
@@ -5,5 +5,5 @@
       <mu1>0.2</mu1>
       <mu2>0.2</mu2>
- 			<kp value="1000000.0" />
+ 			<kp value="100.0" />
 			<kd value="1.0" />
     </gazebo>
@@ -11,5 +11,5 @@
       <mu1>0.2</mu1>
       <mu2>0.2</mu2>
- 			<kp value="1000000.0" />
+ 			<kp value="100.0" />
 			<kd value="1.0" />
     </gazebo>
@@ -17,5 +17,5 @@
       <mu1>0.2</mu1>
       <mu2>0.2</mu2>
- 			<kp value="1000000.0" />
+ 			<kp value="100.0" />
 			<kd value="1.0" />
     </gazebo>
@@ -30,5 +30,5 @@
       <mu1>0.2</mu1>
       <mu2>0.2</mu2>
- 			<kp value="1000000.0" />
+ 			<kp value="100.0" />
 			<kd value="1.0" />
     </gazebo>
@@ -36,5 +36,5 @@
       <mu1>0.2</mu1>
       <mu2>0.2</mu2>
- 			<kp value="1000000.0" />
+ 			<kp value="100.0" />
 			<kd value="1.0" />
     </gazebo>
@@ -42,10 +42,10 @@
       <mu1>0.2</mu1>
       <mu2>0.2</mu2>
- 			<kp value="1000000.0" />
+ 			<kp value="100.0" />
 			<kd value="1.0" />
     </gazebo>
  		<gazebo reference="neck_pan_joint">
 			<kd value="1.0" />
-			<kp value="1000000.0" />
+			<kp value="100.0" />
 			<fudgeFactor value="1.0" />
 			<provideFeedback value="true"/>
@@ -53,5 +53,5 @@
  		<gazebo reference="neck_tilt_joint">
 			<kd value="1.0" />
-			<kp value="1000000.0" />
+			<kp value="100.0" />
 			<fudgeFactor value="1.0" />
 			<provideFeedback value="true"/>
@@ -59,31 +59,31 @@
  		<gazebo reference="eyes_tilt_joint">
 			<kd value="1.0" />
-			<kp value="1000000.0" />
+			<kp value="100.0" />
 			<fudgeFactor value="1.0" />
 			<provideFeedback value="true"/>
 		</gazebo>
  		<gazebo reference="version_joint">
-  		<stopKd value="1000000.0" />
-  		<stopKp value="1000000.0" />
+  		<stopKd value="100.0" />
+  		<stopKp value="100.0" />
 		</gazebo>
  		<!--<gazebo reference="l_eye_version_joint">
-  		<stopKd value="1000000.0" />
-  		<stopKp value="1000000.0" />
+  		<stopKd value="100.0" />
+  		<stopKp value="100.0" />
 		</gazebo>
  		<gazebo reference="r_eye_version_joint">
-  		<stopKd value="1000000.0" />
-  		<stopKp value="1000000.0" />
+  		<stopKd value="100.0" />
+  		<stopKp value="100.0" />
 		</gazebo>-->
  		<gazebo reference="vergence_joint">
-  		<stopKd value="1000000.0" />
-  		<stopKp value="1000000.0" />
+  		<stopKd value="100.0" />
+  		<stopKp value="100.0" />
 		</gazebo>
  		<!--<gazebo reference="l_eye_vergence_joint">
-  		<stopKd value="1000000.0" />
-  		<stopKp value="1000000.0" />
+  		<stopKd value="100.0" />
+  		<stopKp value="100.0" />
 		</gazebo>
  		<gazebo reference="r_eye_vergence_joint">
-  		<stopKd value="1000000.0" />
-  		<stopKp value="1000000.0" />
+  		<stopKd value="100.0" />
+  		<stopKp value="100.0" />
 		</gazebo>-->
 		<gazebo>

File: vizzy_description/urdf/head/head.ros.transmission.xacro (robot description, xacro)
@@ -8,5 +8,5 @@
       <type>transmission_interface/SimpleTransmission</type>
       <joint name="neck_pan_joint">
-        <hardwareInterface>EffortJointInterface</hardwareInterface>
+        <hardwareInterface>VelocityJointInterface</hardwareInterface>
       </joint>
       <actuator name="neck_pan_motor">
@@ -17,5 +17,5 @@
       <type>transmission_interface/SimpleTransmission</type>
       <joint name="neck_tilt_joint">
-        <hardwareInterface>EffortJointInterface</hardwareInterface>
+        <hardwareInterface>VelocityJointInterface</hardwareInterface>
       </joint>
       <actuator name="neck_tilt_motor">
@@ -26,5 +26,5 @@
       <type>transmission_interface/SimpleTransmission</type>
       <joint name="eyes_tilt_joint">
-        <hardwareInterface>EffortJointInterface</hardwareInterface>
+        <hardwareInterface>VelocityJointInterface</hardwareInterface>
       </joint>
       <actuator name="eyes_tilt_motor">
@@ -35,5 +35,5 @@
       <type>transmission_interface/SimpleTransmission</type>
       <joint name="version_joint">
-        <hardwareInterface>EffortJointInterface</hardwareInterface>
+        <hardwareInterface>VelocityJointInterface</hardwareInterface>
       </joint>
       <actuator name="version_motor">
@@ -44,5 +44,5 @@
       <type>transmission_interface/SimpleTransmission</type>
       <joint name="l_eye_version_joint">
-        <hardwareInterface>EffortJointInterface</hardwareInterface>
+        <hardwareInterface>VelocityJointInterface</hardwareInterface>
       </joint>
       <actuator name="l_eye_version_motor">
@@ -53,5 +53,5 @@
       <type>transmission_interface/SimpleTransmission</type>
       <joint name="r_eye_version_joint">
-        <hardwareInterface>EffortJointInterface</hardwareInterface>
+        <hardwareInterface>VelocityJointInterface</hardwareInterface>
       </joint>
       <actuator name="r_eye_version_motor">
@@ -62,5 +62,5 @@
       <type>transmission_interface/SimpleTransmission</type>
       <joint name="vergence_joint">
-        <hardwareInterface>EffortJointInterface</hardwareInterface>
+        <hardwareInterface>VelocityJointInterface</hardwareInterface>
       </joint>
       <actuator name="vergence_motor">
@@ -71,5 +71,5 @@
       <type>transmission_interface/SimpleTransmission</type>
       <joint name="l_eye_vergence_joint">
-        <hardwareInterface>EffortJointInterface</hardwareInterface>
+        <hardwareInterface>VelocityJointInterface</hardwareInterface>
       </joint>
       <actuator name="l_eye_vergence_motor">
@@ -80,5 +80,5 @@
       <type>transmission_interface/SimpleTransmission</type>
       <joint name="r_eye_vergence_joint">
-        <hardwareInterface>EffortJointInterface</hardwareInterface>
+        <hardwareInterface>VelocityJointInterface</hardwareInterface>
       </joint>
       <actuator name="r_eye_vergence_motor">

File: vizzy_description/urdf/head/head.ros.urdf.xacro (robot description, xacro)
@@ -60,5 +60,5 @@
     <axis
       xyz="0 0 1" />
-    <limit lower="-0.925024504" upper="0.925024504" effort="10.0" velocity="3" />
+    <limit lower="-0.925024504" upper="0.925024504" effort="10.0" velocity="5.0" />
     <dynamics damping="0.1" friction="0.1" />
   </joint>
@@ -115,5 +115,5 @@
     <axis
       xyz="0 0 1" />
-    <limit lower="-0.314159265" upper="0.645771823" effort="100.0" velocity="1.0" />
+    <limit lower="-0.314159265" upper="0.645771823" effort="100.0" velocity="5.0" />
     <dynamics damping="10.0" friction="1000000.0" />
   </joint>
@@ -170,5 +170,5 @@
     <axis
       xyz="0 0 1" />
-    <limit lower="-0.663225116" upper="0.663225116" effort="10.0" velocity="3" />
+    <limit lower="-0.663225116" upper="0.663225116" effort="10.0" velocity="5.0" />
     <dynamics damping="0.1" friction="10.0" />
   </joint>

File: vizzy_description/urdf/torso/torso.transmission.xacro (robot description, xacro)
@@ -8,5 +8,5 @@
       <type>transmission_interface/SimpleTransmission</type>
       <joint name="waist_joint">
-        <hardwareInterface>EffortJointInterface</hardwareInterface>
+        <hardwareInterface>VelocityJointInterface</hardwareInterface>
       </joint>
       <actuator name="waist_motor">

Commit message: added new move group for eyes and adjusted control parameters

File: vizzy_description/plugins/ros.gazebo.xacro (robot description, xacro)
@@ -35,6 +35,6 @@
           <horizontal_fov>1.4912</horizontal_fov>
           <image>
-            <width>320</width>
-            <height>240</height>
+            <width>500</width>
+            <height>500</height>
             <!--<width>100</width>
             <height>100</height>-->

File: vizzy_description/urdf/head/head.ros.gazebo.xacro (robot description, xacro)
@@ -21,4 +21,8 @@
     </gazebo>
     <gazebo reference="version_link">
+      <mu1>0.2</mu1>
+      <mu2>0.2</mu2>
+ 			<kp value="1.0" />
+			<kd value="1.0" />
     </gazebo>
     <gazebo reference="r_eye_version_link">
@@ -30,5 +34,5 @@
       <mu1>0.2</mu1>
       <mu2>0.2</mu2>
- 			<kp value="1000000.0" />
+ 			<kp value="1.0" />
 			<kd value="1.0" />
     </gazebo>

File: vizzy_description/urdf/head/head.ros.urdf.xacro (robot description, xacro)
@@ -209,5 +209,5 @@
 			<origin xyz="0 0 0"
       rpy="0.0 0.0 0" />
-			<mass value="0.1"/>
+			<mass value="0.01"/>
 			<inertia
 				ixx="0.001" ixy="0.0" ixz="0.0"
@@ -220,5 +220,5 @@
     <child link="version_link" />
     <axis  xyz="0 0 1" />
-    <limit lower="-0.698131" upper="0.698131" effort="10.0" velocity="0.2" />
+    <limit lower="-0.698131" upper="0.698131" effort="10.0" velocity="5.0" />
     <dynamics damping="1.0" friction="0.7" />
   </joint>
@@ -248,5 +248,5 @@
 			upper="1.0"
       effort="1000.0"
-      velocity="0.2" />
+      velocity="5.0" />
     <dynamics damping="0.1" friction="0.1" />
     <mimic joint="version_joint" multiplier="1" offset="0"/>
@@ -277,5 +277,5 @@
 			upper="1.0"
       effort="1000.0"
-      velocity="0.2"/>
+      velocity="5.0"/>
     <dynamics damping="0.1" friction="0.1" />
     <mimic joint="version_joint" multiplier="1" offset="0"/>
@@ -284,5 +284,5 @@
  		<inertial>
 			<origin xyz="0 0 0" rpy="0 0 0"/>
-			<mass value="0.1"/>
+			<mass value="0.001"/>
 			<inertia
 				ixx="0.001" ixy="0.0" ixz="0.0"
@@ -295,5 +295,5 @@
     <child link="vergence_link" />
     <axis  xyz="0 0 1" />
-    <limit lower="0.0" upper="0.698131" effort="10.0" velocity="0.2" />
+    <limit lower="0.0" upper="0.698131" effort="10.0" velocity="5.0" />
     <dynamics damping="1.0" friction="0.7" />
   </joint>
@@ -353,5 +353,5 @@
 			upper="1.0"
       effort="1000.0"
-      velocity="0.2"/>
+      velocity="5.0"/>
     <dynamics damping="0.1" friction="0.1" />
     <mimic joint="vergence_joint" multiplier="1" offset="0"/>
@@ -438,5 +438,5 @@
 			upper="1.0"
       effort="1000.0"
-      velocity="0.2" />
+      velocity="5.0" />
     <dynamics damping="0.1" friction="0.1" />
     <mimic joint="vergence_joint" multiplier="-1" offset="0"/>

Commit message: small fixes

File: vizzy_description/plugins/ros.gazebo.xacro (robot description, xacro)
@@ -35,6 +35,6 @@
           <horizontal_fov>1.4912</horizontal_fov>
           <image>
-            <width>500</width>
-            <height>500</height>
+            <width>250</width>
+            <height>250</height>
             <!--<width>320</width>
             <height>240</height>-->

File: vizzy_description/urdf/head/head.ros.urdf.xacro (robot description, xacro)
@@ -114,5 +114,6 @@
     <axis
       xyz="0 0 1" />
-    <limit lower="-0.314159265" upper="0.645771823" effort="100.0" velocity="5.0" />
+    <!--<limit lower="-0.314159265" upper="0.645771823" effort="100.0" velocity="5.0" />-->
+    <limit lower="-0.614159265" upper="0.645771823" effort="100.0" velocity="5.0" />
   </joint>
   <link

File: vizzy_description/urdf/simple_base/base.urdf.xacro (robot description, xacro)
@@ -23,5 +23,5 @@
      <origin xyz="0 0 0.25" rpy="0 0 0" />
      <geometry>
-       <cylinder radius="0.1" length="0.5"/>
+       <cylinder radius="0.05" length="0.25"/>
      </geometry>
      <material name="Cyan">
@@ -32,10 +32,10 @@
      <origin xyz="0 0 0.25" rpy="0 0 0"/>
      <geometry>
-       <cylinder radius="0.1" length="0.5"/>
+       <cylinder radius="0.05" length="0.25"/>
      </geometry>
    </collision>
   </link>
   <joint name="waist_joint" type="fixed">
-    <origin xyz="0 0 0.2" rpy="1.57 0 3.14"/>
+    <origin xyz="0 0 0" rpy="1.57 0 3.14"/>
     <parent link="base_link" />
     <child link="waist_link" />
