Commit message: Fixed Vizzy's slippery in simulation. Replaced old caster wheel with new ones. Active wheels now have single point contacts with the floor. Contacts between all wheels balanced. differential_drive_controller had wrong wheel separation value, which was impacting odometry in simulation.

File: vizzy_description/plugins/ros.gazebo.xacro (robot description, xacro)
@@ -17,5 +17,5 @@
         <leftJoint>r_wheel_joint</leftJoint>
         <rightJoint>l_wheel_joint</rightJoint>
-        <wheelSeparation>0.5380</wheelSeparation>
+        <wheelSeparation>0.490</wheelSeparation>
         <wheelDiameter>0.39628</wheelDiameter>
         <torque>20</torque>

File: vizzy_description/urdf/base/base.gazebo.xacro (robot description, xacro)
@@ -1,4 +1,11 @@
 <?xml version="1.0"?>
 <robot xmlns:xacro="http://ros.org/wiki/xacro">
+  <!-- Properties -->
+  <xacro:property name="caster_ball_radius" value="0.05" />
+  <xacro:property name="caster_ball_mass" value="0.870"/>
+  <!-- Materials -->
+  <material name="white">
+    <color rgba="1 1 1 1"/>
+  </material>
   <!-- Load full inertial and collision model or a simplified model -->
   <xacro:arg name="use_full_gazebo_model" default="false"/>
@@ -58,58 +65,40 @@
   </xacro:macro>
   <!-- Caster wheels -->
-  <xacro:macro name="vizzy_caster_wheel_base_link_inertial">
-    <inertial>
-      <origin
-        xyz="-0.0118 0.0084 0.083"
-        rpy="0 0 0" />
-      <mass
-        value="0.4" />
-      <inertia
-        ixx="0.00375" ixy="0.0" ixz="0.0"
-        iyy="0.00375" iyz="0.0"
-        izz="0.00375" />
-    </inertial>
+  <xacro:macro name="gazebo_vizzy_caster_wheel_link" params="name">
+    <link name="${name}_caster_wheel_link">
+      <visual>
+        <geometry>
+          <sphere radius="${caster_ball_radius}"/>
+        </geometry>
+        <material name="light_gray_3"/>
+      </visual>
+      <collision>
+        <geometry>
+          <sphere radius="${caster_ball_radius}"/>
+        </geometry>
+      </collision>
+      <xacro:sphere_inertia m="${caster_ball_mass}" r="${caster_ball_radius}"/>
+    </link>
+    <gazebo reference="${name}_caster_wheel_link">
+      <material>Gazebo/Grey</material>
+      <mu1 value="0.0"/>
+      <mu2 value="0.0"/>
+      <kp  value="10000000.0" />
+      <kd  value="100000.0" />
+    </gazebo>
   </xacro:macro>
-  <xacro:macro name="vizzy_caster_wheel_base_link_collision">
-    <collision>
-      <origin
-        xyz="0 0 0.05"
-        rpy="0 0 0" />
-      <geometry>
-         <cylinder length="0.02" radius="0.01"/>
-      </geometry>
-    </collision>
+  <xacro:macro name="gazebo_vizzy_caster_wheel_joint" params="name parent child origin">
+    <joint name="${name}_caster_wheel_link" type="fixed">
+      <parent link="${parent}"/>
+      <child link="${child}"/>
+      <origin xyz="${origin}"/>
+    </joint>
   </xacro:macro>
-  <xacro:macro name="vizzy_caster_wheel_link_inertial">
-    <inertial>
-      <origin
-        xyz="0 0 0"
-        rpy="0 0 0" />
-      <mass
-        value="0.5" />
-      <xacro:cylinder_inertia
-        m="0.5"
-        r="0.0491365"
-        h="0.02"/>
-    </inertial>
-  </xacro:macro>
-  <xacro:macro name="vizzy_caster_wheel_link_collision">
-    <collision>
-      <origin
-        xyz="0 0 0"
-        rpy="0 0 0"/>
-      <geometry>
-        <cylinder length="0.02" radius="0.0491365"/>
-      </geometry>
-    </collision>
-  </xacro:macro>
-  <xacro:macro name="gazebo_vizzy_caster_wheel_link_surface"
-    params="prefix">
-    <gazebo reference="${prefix}_wheel_link">
-      <mu1 value="1.0" />
-      <mu2 value="1.0" />
-      <kp  value="1000000.0" />
-      <kd  value="1.0" />
-    </gazebo>
+  <xacro:macro name="gazebo_vizzy_caster_wheel" params="name parent origin">
+    <xacro:gazebo_vizzy_caster_wheel_link name="${name}"/>
+    <xacro:gazebo_vizzy_caster_wheel_joint name="${name}"
+      parent="${parent}"
+      child="${name}_caster_wheel_link"
+      origin="${origin}"/>
   </xacro:macro>
   <!-- Active wheels -->
@@ -135,5 +124,5 @@
         rpy="${rpy}" />
       <geometry>
-        <cylinder length="0.06" radius="0.19814"/>
+        <cylinder length="0.001" radius="0.19814"/>
       </geometry>
    </collision>
@@ -142,8 +131,9 @@
     params="prefix">
     <gazebo reference="${prefix}_wheel_link" >
-      <mu1 value="1.0" />
-      <mu2 value="1.0" />
-      <kp  value="1000000.0" />
-      <kd  value="1.0" />
+      <mu1 value="100000.0" />
+      <mu2 value="100000.0" />
+      <maxContacts value="1" />
+      <kp  value="10000000.0" />
+      <kd  value="100000.0" />
     </gazebo>
   </xacro:macro>

File: vizzy_description/urdf/base/base.transmission.xacro (robot description, xacro)
@@ -5,40 +5,4 @@
        xmlns:xacro="http://ros.org/wiki/xacro">
   <xacro:macro name="base_transmissions">
-    <transmission name="f_wheel_transmission">
-      <type>transmission_interface/SimpleTransmission</type>
-      <joint name="f_wheel_joint">
-        <hardwareInterface>hardware_interface/EffortJointInterface</hardwareInterface>
-      </joint>
-      <actuator name="f_wheel_motor">
-        <mechanicalReduction>1</mechanicalReduction>
-      </actuator>
-    </transmission>
-    <transmission name="f_wheel_base_transmission">
-      <type>transmission_interface/SimpleTransmission</type>
-      <joint name="f_wheel_base_joint">
-        <hardwareInterface>hardware_interface/EffortJointInterface</hardwareInterface>
-      </joint>
-      <actuator name="f_wheel_base_motor">
-        <mechanicalReduction>1</mechanicalReduction>
-      </actuator>
-    </transmission>
-    <transmission name="b_wheel_transmission">
-      <type>transmission_interface/SimpleTransmission</type>
-      <joint name="b_wheel_joint">
-        <hardwareInterface>hardware_interface/EffortJointInterface</hardwareInterface>
-      </joint>
-      <actuator name="b_wheel_motor">
-        <mechanicalReduction>1</mechanicalReduction>
-      </actuator>
-    </transmission>
-    <transmission name="b_wheel_base_transmission">
-      <type>transmission_interface/SimpleTransmission</type>
-      <joint name="b_wheel_base_joint">
-        <hardwareInterface>hardware_interface/EffortJointInterface</hardwareInterface>
-      </joint>
-      <actuator name="b_wheel_base_motor">
-        <mechanicalReduction>1</mechanicalReduction>
-      </actuator>
-    </transmission>
     <transmission name="r_wheel_transmission">
       <type>transmission_interface/SimpleTransmission</type>

File: vizzy_description/urdf/base/base.urdf.xacro (robot description, xacro)
@@ -40,113 +40,11 @@
     <xacro:gazebo_vizzy_base_link_surface/>
     <!-- Back (rear) caster wheel -->
-    <link name="b_wheel_base_link">
-      <xacro:vizzy_caster_wheel_base_link_inertial/>
-      <visual>
-        <origin
-          xyz="-0.0118 0.0084 0.083"
-          rpy="0 0 0"/>
-        <geometry>
-          <mesh
-            filename="package://vizzy_description/meshes/base/b_wheel_base.dae"/>
-        </geometry>
-        <material name="light_gray_3"/>
-      </visual>
-      <xacro:vizzy_caster_wheel_base_link_collision/>
-    </link>
-    <joint name="b_wheel_base_joint"
-      type="continuous">
-      <origin
-        xyz="0.43986 0.001 0.1483"
-        rpy="${M_PI} 0 0"/>
-      <parent
-        link="base_link"/>
-      <child
-        link="b_wheel_base_link"/>
-      <axis
-        xyz="0 0 1"/>
-    </joint>
-    <link name="b_wheel_link">
-      <xacro:vizzy_caster_wheel_link_inertial/>
-      <visual>
-        <origin
-          xyz="0 0 0"
-          rpy="0 0 0"/>
-        <geometry>
-          <mesh
-            filename="package://vizzy_description/meshes/base/caster_wheel.dae"/>
-        </geometry>
-        <material name="light_gray_3"/>
-      </visual>
-      <xacro:vizzy_caster_wheel_link_collision/>
-    </link>
-    <joint name="b_wheel_joint"
-      type="continuous">
-      <origin
-        xyz="-0.030027 0.020142 0.138923486"
-        rpy="-1.5708 0.83904 2.5507"/>
-      <parent
-        link="b_wheel_base_link"/>
-      <child
-        link="b_wheel_link"/>
-      <axis
-        xyz="0 0 1"/>
-    </joint>
-    <xacro:gazebo_vizzy_caster_wheel_link_surface
-      prefix="b"/>
+    <xacro:gazebo_vizzy_caster_wheel name="b"
+      parent="base_link"
+      origin="0.43986 0 0.010" />
     <!-- Front caster wheel -->
-    <link name="f_wheel_base_link">
-      <xacro:vizzy_caster_wheel_base_link_inertial/>
-      <visual>
-        <origin
-          xyz="-0.0118 0.0084 0.083"
-          rpy="0 0 0"/>
-        <geometry>
-          <mesh
-            filename="package://vizzy_description/meshes/base/f_wheel_base.dae"/>
-        </geometry>
-        <material name="light_gray_3"/>
-      </visual>
-      <xacro:vizzy_caster_wheel_base_link_collision/>
-    </link>
-    <joint name="f_wheel_base_joint"
-      type="continuous">
-      <origin
-        xyz="-0.060139 0.001 0.1483"
-        rpy="${M_PI} 0 0"/>
-      <parent
-        link="base_link"/>
-      <child
-        link="f_wheel_base_link"/>
-      <axis
-        xyz="0 0 1"/>
-    </joint>
-    <link name="f_wheel_link">
-      <xacro:vizzy_caster_wheel_link_inertial/>
-      <visual>
-        <origin
-          xyz="0 0 0"
-          rpy="0 0 0"/>
-        <geometry>
-          <mesh
-            filename="package://vizzy_description/meshes/base/caster_wheel.dae"/>
-        </geometry>
-        <material name="light_gray_3"/>
-      </visual>
-      <xacro:vizzy_caster_wheel_link_collision/>
-    </link>
-    <joint name="f_wheel_joint"
-      type="continuous">
-      <origin
-        xyz="-0.0300271872634975 0.0201420335543447 0.138923486"
-        rpy="-1.5707963267949 0.83904346430428 2.5507386456365"/>
-      <parent
-        link="f_wheel_base_link"/>
-      <child
-        link="f_wheel_link"/>
-      <axis
-        xyz="0 0 1"/>
-    </joint>
-    <xacro:gazebo_vizzy_caster_wheel_link_surface
-      prefix="f"/>
+    <xacro:gazebo_vizzy_caster_wheel name="f"
+      parent="base_link"
+      origin="-0.060139 0 0.010" />
     <!-- Right wheel -->
     <link name="r_wheel_link">

File: vizzy_description/urdf/common.urdf.xacro (robot description, xacro)
@@ -35,4 +35,12 @@
       izz="${m*r*r/2}"/>
   </xacro:macro>
+  <xacro:macro name="sphere_inertia" params="m r">
+    <inertial>
+      <mass value="${m}" />
+      <inertia ixx="${2.0 / 5.0 * m * r * r}" ixy="0.0" ixz="0.0"
+               iyy="${2.0 / 5.0 * m * r * r}" iyz="0.0"
+               izz="${2.0 / 5.0 * m * r * r}" />
+    </inertial>
+  </xacro:macro>
   <!-- Colors -->
   <material name="light_grey">
