Commit message: Realsense working on Gazebo. Tested on ROS Melodic

File: vizzy_description/urdf/sensors/_d435.urdf.xacro (robot description, xacro)
@@ -7,5 +7,7 @@
 -->
 <robot name="sensor_d435" xmlns:xacro="http://ros.org/wiki/xacro">
-  <xacro:macro name="sensor_d435" params="name parent *origin">
+  <!--File includes-->
+  <xacro:include filename="$(find vizzy_description)/urdf/sensors/_d435.gazebo.xacro"/>
+  <xacro:macro name="sensor_d435" params="name parent topics_ns:=realsense *origin">
     <xacro:property name="M_PI" value="3.1415926535897931" />
     <!-- The following values are approximate, and the camera node
@@ -116,4 +118,6 @@
     </joint>
     <link name="${name}_color_optical_frame"/>
+    <!-- Realsense Gazebo Plugin -->
+    <xacro:gazebo_d435 camera_name="${name}" reference_link="${name}_link" topics_ns="${topics_ns}" depth_optical_frame="${name}_depth_optical_frame" color_optical_frame="${name}_color_optical_frame" infrared1_optical_frame="${name}_left_ir_optical_frame" infrared2_optical_frame="${name}_right_ir_optical_frame"/>
   </xacro:macro>
 </robot>

Commit message: [d435] Corrected link to d435 mesh [real_robot] Added google speech interface and super-service batteries state service

File: vizzy_description/urdf/sensors/_d435.urdf.xacro (robot description, xacro)
@@ -48,5 +48,5 @@
         <geometry>
           <!-- <box size="${d435_cam_width} ${d435_cam_height} ${d435_cam_depth}"/> -->
-	  <mesh filename="package://realsense2_camera/meshes/d435.dae" />
+	        <mesh filename="package://realsense2_description/meshes/d435.dae" />
           <!--<mesh filename="package://realsense2_camera/meshes/d435/d435.dae" />-->
         </geometry>
